File: mainBoard/mainBoard.kicad_pcb (KiCad board)
At the start: 4 copper layers, 0 parts

Commit message: Schematic Capture should be complete, ready for PCB
Parts:
- added BZ1: Buzzer, Buzzer_Beeper:Buzzer_12x9.5RM7.6, F.Cu at (183.3, 65.8)
- added C1: 10uF, Capacitor_SMD:C_0805_2012Metric_Pad1.18x1.45mm_HandSolder, F.Cu at (140.1, 83.7)
- added C10: 20pF, Capacitor_SMD:C_0402_1005Metric_Pad0.74x0.62mm_HandSolder, F.Cu at (172.8, 114.4)
- added C11: 100nF, Capacitor_SMD:C_0603_1608Metric_Pad1.08x0.95mm_HandSolder, F.Cu at (154.3, 119.2)
- added C12: 2.2uF Low ESR, Capacitor_SMD:C_0805_2012Metric_Pad1.18x1.45mm_HandSolder, F.Cu at (173.6, 102.5)
- added C13: 1uF, Capacitor_SMD:C_0805_2012Metric_Pad1.18x1.45mm_HandSolder, F.Cu at (173.6, 105.5)
- added C14: 100nF, Capacitor_SMD:C_0603_1608Metric_Pad1.08x0.95mm_HandSolder, F.Cu at (154.3, 121.7)
- added C15: 100nF, Capacitor_SMD:C_0603_1608Metric_Pad1.08x0.95mm_HandSolder, F.Cu at (154.3, 124.2)
- added C16: 100nF, Capacitor_SMD:C_0603_1608Metric_Pad1.08x0.95mm_HandSolder, F.Cu at (158.7, 116.7)
- added C17: 100nF, Capacitor_SMD:C_0603_1608Metric_Pad1.08x0.95mm_HandSolder, F.Cu at (158.7, 119.2)
- added C18: 100nF, Capacitor_SMD:C_0603_1608Metric_Pad1.08x0.95mm_HandSolder, F.Cu at (158.7, 121.7)
- added C19: 10nF 250V, Capacitor_SMD:C_1812_4532Metric_Pad1.57x3.40mm_HandSolder, F.Cu at (217.8, 107.9)
- added C2: 1uF, Capacitor_SMD:C_0805_2012Metric_Pad1.18x1.45mm_HandSolder, F.Cu at (140.1, 86.7)
- added C20: 1uF X7R, Capacitor_SMD:C_0603_1608Metric_Pad1.08x0.95mm_HandSolder, F.Cu at (133.4, 116.6)
- added C21: 100nF, Capacitor_SMD:C_0805_2012Metric_Pad1.18x1.45mm_HandSolder, F.Cu at (138.0, 126.3)
- added C22: 100nF, Capacitor_SMD:C_0805_2012Metric_Pad1.18x1.45mm_HandSolder, F.Cu at (138.0, 129.3)
- added C3: 10uF, Capacitor_SMD:C_0805_2012Metric_Pad1.18x1.45mm_HandSolder, F.Cu at (140.1, 89.7)
- added C4: 47uF, Capacitor_THT:C_Radial_D5.0mm_H5.0mm_P2.00mm, F.Cu at (163.6, 93.2)
- added C5: 1uF, Capacitor_SMD:C_0805_2012Metric_Pad1.18x1.45mm_HandSolder, F.Cu at (140.1, 92.7)
- added C6: 100nF, Capacitor_SMD:C_0603_1608Metric_Pad1.08x0.95mm_HandSolder, F.Cu at (144.7, 83.4)
- added C7: 10uF, Capacitor_SMD:C_0805_2012Metric_Pad1.18x1.45mm_HandSolder, F.Cu at (140.1, 95.7)
- added C8: 100nF, Capacitor_SMD:C_0603_1608Metric_Pad1.08x0.95mm_HandSolder, F.Cu at (154.3, 116.7)
- added C9: 20pF, Capacitor_SMD:C_0402_1005Metric_Pad0.74x0.62mm_HandSolder, F.Cu at (172.8, 112.4)
- added D1: RED, LED_SMD:LED_0603_1608Metric_Pad1.05x0.95mm_HandSolder, F.Cu at (170.0, 91.2)
- added D2: RED, LED_SMD:LED_0603_1608Metric_Pad1.05x0.95mm_HandSolder, F.Cu at (170.0, 93.8)
- added D3: RED, LED_SMD:LED_0603_1608Metric_Pad1.05x0.95mm_HandSolder, F.Cu at (168.8, 111.9)
- added D4: RED, LED_SMD:LED_0603_1608Metric_Pad1.05x0.95mm_HandSolder, F.Cu at (216.3, 116.7)
- added D5: T2035T-8G-RT, Package_TO_SOT_SMD:TO-263-2, F.Cu at (215.8, 99.2)
- added D6: 1N5819HW-7-F, Diode_SMD:D_SOD-123, F.Cu at (219.2, 45.1)
- added D7: 1N5819HW-7-F, Diode_SMD:D_SOD-123, F.Cu at (219.2, 48.5)
- added D8: 1N5819HW-7-F, Diode_SMD:D_SOD-123, F.Cu at (219.2, 51.8)
- added F1: 1A, Fuse:Fuseholder_Clip-5x20mm_Littelfuse_100_Inline_P20.50x4.60mm_D1.30mm_Horizontal, F.Cu at (139.6, 66.3)
- added F2: 20A, Fuse:Fuseholder_Clip-6.3x32mm_Littelfuse_122_Inline_P34.21x7.62mm_D2.54mm_Horizontal, F.Cu at (182.9, 88.3)
- added FB1: WLBD2012HCU601TH, Inductor_SMD:L_0805_2012Metric_Pad1.05x1.20mm_HandSolder, F.Cu at (174.7, 91.3)
- added H1: MountingHole, MountingHole:MountingHole_3mm, F.Cu at (184.2, 96.8)
- added H2: MountingHole, MountingHole:MountingHole_3mm, F.Cu at (184.2, 104.4)
- added H3: MountingHole, MountingHole:MountingHole_3mm, F.Cu at (184.2, 111.9)
- added H4: MountingHole, MountingHole:MountingHole_3mm, F.Cu at (184.2, 119.5)
- added J1: 1366005, PhoenixContact_SPTA:SPTA-THR 2.53-5.0 P26, F.Cu at (169.8, 72.9)
- added J10: Conn_01x07, Connector_JST:JST_XH_B7B-XH-A_1x07_P2.50mm_Vertical, F.Cu at (183.8, 39.0)
- added J11: Conn_01x04, Connector_JST:JST_XH_B4B-XH-A_1x04_P2.50mm_Vertical, F.Cu at (183.8, 46.8)
- added J12: Conn_01x04, Connector_JST:JST_XH_B4B-XH-A_1x04_P2.50mm_Vertical, F.Cu at (183.8, 54.6)
- added J13: Conn_01x05, Connector_JST:JST_XH_B5B-XH-A_1x05_P2.50mm_Vertical, F.Cu at (205.8, 39.0)
- added J14: Conn_02x05_Odd_Even, Connector_IDC:IDC-Header_2x05_P2.54mm_Vertical, F.Cu at (200.1, 49.5)
- added J15: Conn_01x06, Connector_PinHeader_2.54mm:PinHeader_1x06_P2.54mm_Vertical, F.Cu at (214.0, 61.3)
- added J16: Conn_01x08, Connector_PinHeader_2.54mm:PinHeader_1x08_P2.54mm_Vertical, F.Cu at (218.6, 61.3)
- added J2: Conn_01x02, TerminalBlock_Phoenix:TerminalBlock_Phoenix_MKDS-1,5-2-5.08_1x02_P5.08mm_Horizontal, F.Cu at (129.0, 68.8)
- added J3: Conn_01x02, TerminalBlock_Phoenix:TerminalBlock_Phoenix_MKDS-1,5-2-5.08_1x02_P5.08mm_Horizontal, F.Cu at (129.0, 80.9)
- added J4: Conn_01x03, Connector_JST:JST_XH_B3B-XH-A_1x03_P2.50mm_Vertical, F.Cu at (208.5, 123.5)
- added J5: 1366005, PhoenixContact_SPTA:SPTA-THR 2.53-5.0 P26, F.Cu at (196.5, 95.8)
- added J6: 4DB-P108-02, 4DB_P108_02:CONN_4DB-P108-02_TEC, F.Cu at (131.5, 104.1)
- added J7: Conn_01x02, Connector_JST:JST_XH_B2B-XH-A_1x02_P2.50mm_Vertical, F.Cu at (210.3, 46.8)
- added J8: Conn_01x02, Connector_JST:JST_XH_B2B-XH-A_1x02_P2.50mm_Vertical, F.Cu at (210.3, 54.6)
- added J9: Conn_01x03, Connector_JST:JST_XH_B3B-XH-A_1x03_P2.50mm_Vertical, F.Cu at (198.3, 69.2)
- added JP1: Jumper_2_Open, Connector_PinHeader_2.54mm:PinHeader_1x02_P2.54mm_Vertical, F.Cu at (149.1, 84.5)
- added JP2: Jumper_2_Open, Connector_PinHeader_2.54mm:PinHeader_1x02_P2.54mm_Vertical, F.Cu at (153.7, 84.5)
- added JP3: Jumper_2_Open, Jumper:SolderJumper-2_P1.3mm_Open_TrianglePad1.0x1.5mm, F.Cu at (147.9, 102.7)
- added JP4: Jumper_2_Open, Jumper:SolderJumper-2_P1.3mm_Open_TrianglePad1.0x1.5mm, F.Cu at (197.0, 75.4)
- added JP5: Jumper_2_Open, Jumper:SolderJumper-2_P1.3mm_Open_TrianglePad1.0x1.5mm, F.Cu at (197.0, 79.0)
- added NT1: NetTie_2, NetTie:NetTie-2_SMD_Pad0.5mm, F.Cu at (173.5, 93.4)
- added PS1: IRM-10-5, Converter_ACDC:Converter_ACDC_MeanWell_IRM-10-xx_THT, F.Cu at (130.0, 47.6)
- added Q1: IRLML6244TRPBF, Package_TO_SOT_SMD:SOT-23, F.Cu at (173.7, 109.2)
- added Q2: IRLML6244TRPBF, Package_TO_SOT_SMD:SOT-23, F.Cu at (209.3, 61.2)
- added Q3: IRLML6244TRPBF, Package_TO_SOT_SMD:SOT-23, F.Cu at (209.3, 65.7)
- added Q4: IRLML6244TRPBF, Package_TO_SOT_SMD:SOT-23, F.Cu at (209.3, 70.2)
- added Q5: IRLML6244TRPBF, Package_TO_SOT_SMD:SOT-23, F.Cu at (209.3, 74.6)
- added R1: 10k, Resistor_SMD:R_0603_1608Metric_Pad0.98x0.95mm_HandSolder, F.Cu at (144.7, 85.9)
- added R10: 330, Resistor_SMD:R_0603_1608Metric_Pad0.98x0.95mm_HandSolder, F.Cu at (216.2, 114.1)
- added R11: 330, Resistor_SMD:R_2512_6332Metric_Pad1.40x3.35mm_HandSolder, F.Cu at (209.6, 107.8)
- added R12: 330, Resistor_SMD:R_2512_6332Metric_Pad1.40x3.35mm_HandSolder, F.Cu at (209.6, 112.8)
- added R13: 39, Resistor_SMD:R_2512_6332Metric_Pad1.40x3.35mm_HandSolder, F.Cu at (209.6, 117.7)
- added R14: 100k, Resistor_SMD:R_0603_1608Metric_Pad0.98x0.95mm_HandSolder, F.Cu at (133.4, 119.1)
- added R15: 100k, Resistor_SMD:R_0603_1608Metric_Pad0.98x0.95mm_HandSolder, F.Cu at (133.4, 121.6)
- added R16: 560, Resistor_SMD:R_0603_1608Metric_Pad0.98x0.95mm_HandSolder, F.Cu at (133.4, 124.1)
- added R17: TC33X-2-102E, Potentiometer_SMD:Potentiometer_Bourns_TC33X_Vertical, F.Cu at (138.7, 117.7)
- added R18: 280k, Resistor_SMD:R_0603_1608Metric_Pad0.98x0.95mm_HandSolder, F.Cu at (133.4, 126.6)
- added R19: TC33X-2-104E, Potentiometer_SMD:Potentiometer_Bourns_TC33X_Vertical, F.Cu at (138.7, 122.4)
- added R2: 220, Resistor_SMD:R_0603_1608Metric_Pad0.98x0.95mm_HandSolder, F.Cu at (144.7, 88.4)
- added R20: 1k, Resistor_SMD:R_0603_1608Metric_Pad0.98x0.95mm_HandSolder, F.Cu at (133.4, 129.1)
- added R21: 1k, Resistor_SMD:R_0603_1608Metric_Pad0.98x0.95mm_HandSolder, F.Cu at (223.1, 60.3)
- added R22: 1k, Resistor_SMD:R_0603_1608Metric_Pad0.98x0.95mm_HandSolder, F.Cu at (223.1, 62.8)
- added R23: 1k, Resistor_SMD:R_0603_1608Metric_Pad0.98x0.95mm_HandSolder, F.Cu at (223.1, 65.3)
- added R24: 220, Resistor_SMD:R_0603_1608Metric_Pad0.98x0.95mm_HandSolder, F.Cu at (223.1, 67.8)
- added R25: 10k, Resistor_SMD:R_0603_1608Metric_Pad0.98x0.95mm_HandSolder, F.Cu at (223.1, 70.3)
- added R26: 10k, Resistor_SMD:R_0603_1608Metric_Pad0.98x0.95mm_HandSolder, F.Cu at (223.1, 72.8)
- added R27: 10k, Resistor_SMD:R_0603_1608Metric_Pad0.98x0.95mm_HandSolder, F.Cu at (223.1, 75.3)
- added R28: 10k, Resistor_SMD:R_0603_1608Metric_Pad0.98x0.95mm_HandSolder, F.Cu at (223.1, 77.8)
- added R29: 1k, Resistor_SMD:R_0603_1608Metric_Pad0.98x0.95mm_HandSolder, F.Cu at (223.1, 80.4)
- added R3: 330, Resistor_SMD:R_0603_1608Metric_Pad0.98x0.95mm_HandSolder, F.Cu at (144.7, 91.0)
- added R4: 10k, Resistor_SMD:R_0603_1608Metric_Pad0.98x0.95mm_HandSolder, F.Cu at (158.7, 124.2)
- added R5: 10k, Resistor_SMD:R_0603_1608Metric_Pad0.98x0.95mm_HandSolder, F.Cu at (163.0, 116.7)
- added R6: 220, Resistor_SMD:R_0603_1608Metric_Pad0.98x0.95mm_HandSolder, F.Cu at (163.0, 119.2)
- added R7: 10k, Resistor_SMD:R_0603_1608Metric_Pad0.98x0.95mm_HandSolder, F.Cu at (163.0, 121.7)
- added R8: 220, Resistor_SMD:R_0603_1608Metric_Pad0.98x0.95mm_HandSolder, F.Cu at (163.0, 124.2)
- added R9: 330, Resistor_SMD:R_0603_1608Metric_Pad0.98x0.95mm_HandSolder, F.Cu at (216.2, 111.6)
- added RV1: TMOV20RP150E, TMOV20RP150E:TMOV20RP150E, F.Cu at (145.7, 74.7)
- added SW1: SW_SPST, TerminalBlock_Phoenix:TerminalBlock_Phoenix_MKDS-1,5-2-5.08_1x02_P5.08mm_Horizontal, F.Cu at (129.0, 93.1)
- added SW2: SW_SPDT, Connector_PinHeader_2.54mm:PinHeader_1x03_P2.54mm_Vertical, F.Cu at (168.9, 103.2)
- added SW3: SW_Push, Button_Switch_THT:SW_PUSH_6mm_H4.3mm, F.Cu at (167.2, 124.1)
- added TP1: TestPoint, TestPoint:TestPoint_Keystone_5019_Miniature, F.Cu at (128.3, 117.3)
- added TP2: TestPoint, TestPoint:TestPoint_Keystone_5019_Miniature, F.Cu at (128.3, 121.2)
- added TP3: TestPoint, TestPoint:TestPoint_Keystone_5019_Miniature, F.Cu at (128.3, 125.2)
- added TP4: TestPoint, TestPoint:TestPoint_Keystone_5019_Miniature, F.Cu at (128.3, 129.1)
- added U1: MCP1727T-3302E/SN, Package_SO:SOIC-8_3.9x4.9mm_P1.27mm, F.Cu at (151.1, 92.7)
- added U2: STM32F401RETx, Package_QFP:LQFP-64_10x10mm_P0.5mm, F.Cu at (159.4, 108.2)
- added U3: DS18B20+, Connector_JST:JST_PH_B3B-PH-K_1x03_P2.00mm_Vertical, F.Cu at (190.9, 124.8)
- added U4: MOC3083S-TA1, Package_DIP:SMDIP-6_W9.53mm, F.Cu at (194.5, 117.5)
- added U5: DS18B20+, Package_TO_SOT_THT:TO-92_Inline, F.Cu at (143.7, 125.1)
- added U6: OPA333AIDCKT, Package_SO:SOIC-8_3.9x4.9mm_P1.27mm, F.Cu at (145.9, 118.7)
- added Y1: ATS240C-E, Crystal:Crystal_HC49-4H_Vertical, F.Cu at (169.3, 118.8)

Commit message: tweak schematic for changes from 6-17-2026
major structural changes, see daily note from obsidian
Parts:
- removed the J13 at (205.8, 39.0)
- removed the J4 at (208.5, 123.5)
- removed the J9 at (198.3, 69.2)
- added ?: , , F.Cu at (317.5, 117.0)
- added ?: , , F.Cu at (541.5, 117.2)
- added ?: , , F.Cu at (317.5, 38.0)
- added ?: , , F.Cu at (541.5, 38.2)
- added ?: , , F.Cu at (396.5, 99.8)
- added ?: , , F.Cu at (499.8, 86.0)
- added C23: 10nF 250V, Capacitor_SMD:C_1812_4532Metric_Pad1.57x3.40mm_HandSolder, F.Cu at (236.2, 118.1)
- added C24: 1uF X7R, Capacitor_SMD:C_0603_1608Metric_Pad1.08x0.95mm_HandSolder, F.Cu at (234.0, 73.4)
- added C25: 100nF, Capacitor_SMD:C_0805_2012Metric_Pad1.18x1.45mm_HandSolder, F.Cu at (266.5, 44.9)
- added C26: 100nF, Capacitor_SMD:C_0805_2012Metric_Pad1.18x1.45mm_HandSolder, F.Cu at (266.5, 47.9)
- added C27: 1uF X7R, Capacitor_SMD:C_0603_1608Metric_Pad1.08x0.95mm_HandSolder, F.Cu at (234.0, 75.9)
- added C28: 100nF, Capacitor_SMD:C_0805_2012Metric_Pad1.18x1.45mm_HandSolder, F.Cu at (266.5, 50.9)
- added C29: 100nF, Capacitor_SMD:C_0805_2012Metric_Pad1.18x1.45mm_HandSolder, F.Cu at (266.5, 53.9)
- added C30: 10uF, Capacitor_SMD:C_0805_2012Metric_Pad1.18x1.45mm_HandSolder, F.Cu at (101.8, 108.5)
- added C31: 1uF, Capacitor_SMD:C_0805_2012Metric_Pad1.18x1.45mm_HandSolder, F.Cu at (101.8, 111.5)
- added C32: 10uF, Capacitor_SMD:C_0805_2012Metric_Pad1.18x1.45mm_HandSolder, F.Cu at (101.8, 114.5)
- added C33: 100nF, Capacitor_SMD:C_0603_1608Metric_Pad1.08x0.95mm_HandSolder, F.Cu at (122.3, 71.8)
- added C34: 22uF, Capacitor_THT:C_Radial_D5.0mm_H11.0mm_P2.00mm, F.Cu at (109.8, 80.3)
- added C35: 22uF, Capacitor_THT:C_Radial_D5.0mm_H11.0mm_P2.00mm, F.Cu at (109.8, 86.9)
- added C7: 10uF, Capacitor_THT:C_Radial_D5.0mm_H11.0mm_P2.00mm, F.Cu at (109.8, 73.8)
- added D10: T2035T-8G-RT, Package_TO_SOT_THT:TO-220-3_Vertical, F.Cu at (244.7, 119.9)
- added D11: RED, LED_SMD:LED_0603_1608Metric_Pad1.05x0.95mm_HandSolder, F.Cu at (106.5, 115.4)
- added D12: RED, LED_SMD:LED_0603_1608Metric_Pad1.05x0.95mm_HandSolder, F.Cu at (120.9, 88.5)
- added D13: 1N5819HW-7-F, Diode_SMD:D_SOD-123, F.Cu at (80.4, 100.8)
- added D9: RED, LED_SMD:LED_0603_1608Metric_Pad1.05x0.95mm_HandSolder, F.Cu at (239.0, 121.8)
- added F3: 10A, Fuse:Fuseholder_Clip-6.3x32mm_Littelfuse_122_Inline_P34.21x7.62mm_D2.54mm_Horizontal, F.Cu at (217.9, 96.1)
- added F4: 3A, Fuse:Fuseholder_Clip-5x20mm_Littelfuse_100_Inline_P20.50x4.60mm_D1.30mm_Horizontal, F.Cu at (62.5, 83.3)
- added H5: MountingHole_Pad, MountingHole:MountingHole_2.7mm, F.Cu at (541.5, 38.2)
- added H6: MountingHole_Pad, MountingHole:MountingHole_2.7mm, F.Cu at (541.5, 117.2)
- added HS1: 530002B02500G, 530002_Heatsinks:53002B02500G, F.Cu at (55.3, 127.0)
- added HS2: 530002B02500G, 530002_Heatsinks:53002B02500G, F.Cu at (55.3, 155.5)
- added J17: Conn_01x02, TerminalBlock_Phoenix:TerminalBlock_Phoenix_MKDS-1,5-2-5.08_1x02_P5.08mm_Horizontal, F.Cu at (81.0, 93.2)
- added J5: 4DB-P108-02, 4DB_P108_02:CONN_4DB-P108-02_TEC, F.Cu at (212.7, 32.5)
- added J8: Conn_01x02, Connector_JST:JST_XH_B2B-XH-A_1x02_P2.50mm_Vertical, F.Cu at (223.8, 71.4)
- added JP6: Jumper_2_Open, Jumper:SolderJumper-2_P1.3mm_Open_TrianglePad1.0x1.5mm, F.Cu at (260.1, 77.3)
- added JP7: Jumper_2_Open, Jumper:SolderJumper-2_P1.3mm_Open_TrianglePad1.0x1.5mm, F.Cu at (260.1, 80.9)
- added JP8: Jumper_2_Open, Connector_PinHeader_2.54mm:PinHeader_1x02_P2.54mm_Vertical, F.Cu at (106.5, 109.3)
- added JP9: Jumper_2_Open, Connector_PinHeader_2.54mm:PinHeader_1x02_P2.54mm_Vertical, F.Cu at (116.3, 84.9)
- added K1: Relay_SPDT, Relay_THT:Relay_SPDT_Finder_36.11, F.Cu at (63.1, 91.0)
- added NT2: NetTie_2, NetTie:NetTie-2_SMD_Pad0.5mm, F.Cu at (100.7, 116.7)
- added Q6: IRLML6244TRPBF, Package_TO_SOT_SMD:SOT-23, F.Cu at (79.9, 104.7)
- added R30: 330, Resistor_SMD:R_0603_1608Metric_Pad0.98x0.95mm_HandSolder, F.Cu at (234.6, 121.8)
- added R31: 330, Resistor_SMD:R_0603_1608Metric_Pad0.98x0.95mm_HandSolder, F.Cu at (234.6, 124.3)
- added R32: 330, Resistor_SMD:R_2512_6332Metric_Pad1.40x3.35mm_HandSolder, F.Cu at (237.0, 103.3)
- added R33: 330, Resistor_SMD:R_2512_6332Metric_Pad1.40x3.35mm_HandSolder, F.Cu at (237.0, 108.2)
- added R34: 39, Resistor_SMD:R_2512_6332Metric_Pad1.40x3.35mm_HandSolder, F.Cu at (237.0, 113.1)
- added R35: 100k, Resistor_SMD:R_0603_1608Metric_Pad0.98x0.95mm_HandSolder, F.Cu at (234.0, 78.4)
- added R36: 100k, Resistor_SMD:R_0603_1608Metric_Pad0.98x0.95mm_HandSolder, F.Cu at (234.0, 80.9)
- added R37: 560, Resistor_SMD:R_0603_1608Metric_Pad0.98x0.95mm_HandSolder, F.Cu at (238.4, 73.4)
- added R38: TC33X-2-102E, Potentiometer_SMD:Potentiometer_Bourns_TC33X_Vertical, F.Cu at (261.1, 45.8)
- added R39: 280k, Resistor_SMD:R_0603_1608Metric_Pad0.98x0.95mm_HandSolder, F.Cu at (238.4, 75.9)
- added R40: TC33X-2-104E, Potentiometer_SMD:Potentiometer_Bourns_TC33X_Vertical, F.Cu at (261.1, 50.5)
- added R41: 1k, Resistor_SMD:R_0603_1608Metric_Pad0.98x0.95mm_HandSolder, F.Cu at (238.4, 78.4)
- added R42: 100k, Resistor_SMD:R_0603_1608Metric_Pad0.98x0.95mm_HandSolder, F.Cu at (238.4, 80.9)
- added R43: 100k, Resistor_SMD:R_0603_1608Metric_Pad0.98x0.95mm_HandSolder, F.Cu at (242.7, 73.4)
- added R44: 560, Resistor_SMD:R_0603_1608Metric_Pad0.98x0.95mm_HandSolder, F.Cu at (242.7, 75.9)
- added R45: TC33X-2-102E, Potentiometer_SMD:Potentiometer_Bourns_TC33X_Vertical, F.Cu at (261.1, 55.3)
- added R46: 280k, Resistor_SMD:R_0603_1608Metric_Pad0.98x0.95mm_HandSolder, F.Cu at (242.7, 78.4)
- added R47: TC33X-2-104E, Potentiometer_SMD:Potentiometer_Bourns_TC33X_Vertical, F.Cu at (261.1, 60.0)
- added R48: 1k, Resistor_SMD:R_0603_1608Metric_Pad0.98x0.95mm_HandSolder, F.Cu at (242.7, 80.9)
- added R49: 10k, Resistor_SMD:R_0603_1608Metric_Pad0.98x0.95mm_HandSolder, F.Cu at (95.5, 113.7)
- added R50: 220, Resistor_SMD:R_0603_1608Metric_Pad0.98x0.95mm_HandSolder, F.Cu at (95.5, 116.2)
- added R51: 52.3k, Resistor_SMD:R_0603_1608Metric_Pad0.98x0.95mm_HandSolder, F.Cu at (122.3, 74.3)
- added R52: 10k, Resistor_SMD:R_0603_1608Metric_Pad0.98x0.95mm_HandSolder, F.Cu at (122.3, 76.8)
- added R53: 330, Resistor_SMD:R_0603_1608Metric_Pad0.98x0.95mm_HandSolder, F.Cu at (122.3, 79.3)
- added R54: 1k, Resistor_SMD:R_0603_1608Metric_Pad0.98x0.95mm_HandSolder, F.Cu at (85.4, 100.4)
- added R55: 10k, Resistor_SMD:R_0603_1608Metric_Pad0.98x0.95mm_HandSolder, F.Cu at (85.4, 102.9)
- added TP10: TestPoint, TestPoint:TestPoint_Keystone_5019_Miniature, F.Cu at (255.1, 49.3)
- added TP11: TestPoint, TestPoint:TestPoint_Keystone_5019_Miniature, F.Cu at (255.1, 53.3)
- added TP12: TestPoint, TestPoint:TestPoint_Keystone_5019_Miniature, F.Cu at (255.1, 57.2)
- added TP13: TestPoint, TestPoint:TestPoint_Keystone_5019_Miniature, F.Cu at (255.1, 61.2)
- added TP14: TestPoint, TestPoint:TestPoint_Keystone_5019_Miniature, F.Cu at (255.1, 65.1)
- added TP15: TestPoint, TestPoint:TestPoint_Keystone_5019_Miniature, F.Cu at (255.1, 69.1)
- added TP16: TestPoint, TestPoint:TestPoint_Keystone_5019_Miniature, F.Cu at (255.1, 73.0)
- added TP17: TestPoint, TestPoint:TestPoint_Pad_4.0x4.0mm, F.Cu at (96.4, 103.4)
- added TP18: TestPoint, TestPoint:TestPoint_Pad_4.0x4.0mm, F.Cu at (96.4, 109.5)
- added TP5: TestPoint, TestPoint:TestPoint_Pad_4.0x4.0mm, F.Cu at (104.3, 72.9)
- added TP6: TestPoint, TestPoint:TestPoint_Pad_4.0x4.0mm, F.Cu at (103.8, 79.9)
- added TP9: TestPoint, TestPoint:TestPoint_Keystone_5019_Miniature, F.Cu at (255.1, 45.4)
- added U10: OPA333AIDCKT, Package_SO:SOIC-8_3.9x4.9mm_P1.27mm, F.Cu at (262.2, 72.3)
- added U11: DS18B20+, Package_TO_SOT_THT:TO-92_Inline, F.Cu at (246.9, 81.2)
- added U12: MCP1727T-3302E/SN, Package_SO:SOIC-8_3.9x4.9mm_P1.27mm, F.Cu at (103.6, 103.7)
- added U13: AP62250WU, Package_TO_SOT_SMD:TSOT-23-6_HandSoldering, F.Cu at (122.1, 85.0)
- added U7: MOC3083S-TA1, Package_DIP:SMDIP-6_W9.53mm, F.Cu at (248.1, 105.4)
- added U8: OPA333AIDCKT, Package_SO:SOIC-8_3.9x4.9mm_P1.27mm, F.Cu at (262.2, 65.8)
- added U9: DS18B20+, Package_TO_SOT_THT:TO-92_Inline, F.Cu at (246.9, 75.4)
- C4: footprint Capacitor_THT:C_Radial_D5.0mm_H5.0mm_P2.00mm -> Capacitor_THT:C_Radial_D5.0mm_H11.0mm_P2.00mm
- D5: footprint Package_TO_SOT_SMD:TO-263-2 -> Package_TO_SOT_THT:TO-220-3_Vertical
- F2: value 20A -> 10A
- H1, H2, H3, H4: value MountingHole -> MountingHole_Pad; footprint MountingHole:MountingHole_3mm -> MountingHole:MountingHole_2.7mm
- J2: value Conn_01x02 -> 1366005; footprint TerminalBlock_Phoenix:TerminalBlock_Phoenix_MKDS-1,5-2-5.08_1x02_P5.08mm_Horizontal -> PhoenixContact_SPTA:SPTA-THR 2.53-5.0 P26
- J3: value Conn_01x02 -> 4DB-P108-02; footprint TerminalBlock_Phoenix:TerminalBlock_Phoenix_MKDS-1,5-2-5.08_1x02_P5.08mm_Horizontal -> 4DB_P108_02:CONN_4DB-P108-02_TEC
- PS1: value IRM-10-5 -> IRM-30-12; footprint Converter_ACDC:Converter_ACDC_MeanWell_IRM-10-xx_THT -> IRM-30:IRM-30_MWU
- R3: value 330 -> 1.2k
- U3: footprint Connector_JST:JST_PH_B3B-PH-K_1x03_P2.00mm_Vertical -> Package_TO_SOT_THT:TO-92_Inline
- Y1: footprint Crystal:Crystal_HC49-4H_Vertical -> Crystal:Crystal_SMD_3225-4Pin_3.2x2.5mm
- moved H4 317.4 mm to (499.8, 86.0)
- moved PS1 228.1 mm to (358.0, 40.5), turned to -90 degrees
- moved H3 212.7 mm to (396.5, 99.8)
- moved D5 173.8 mm to (53.0, 160.0)
- moved H1 145.7 mm to (317.5, 38.0), turned to 180 degrees
- moved H2 133.9 mm to (317.5, 117.0)
- moved J4 108.6 mm to (182.0, -11.8), turned to 180 degrees
- moved J3 104.7 mm to (212.7, 18.1)
- moved J1 89.8 mm to (200.0, -11.8), turned to 180 degrees
- moved J2 87.4 mm to (163.5, -11.5), turned to 180 degrees
- moved U3 14.3 mm to (185.5, 138.0)
- moved C11 13.1 mm to (142.7, 125.1)
- moved C15 13.1 mm to (142.7, 130.1)
- moved C17 13.1 mm to (147.0, 125.1)
- moved C21 13.1 mm to (126.3, 132.2)
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- renumbered J11 to J10, J12 to J11, J14 to J13, J15 to J14, J16 to J15, J6 to J16, J5 to J4, J7 to J6, J8 to J7, J10 to J9
Connections:
- net /Project Architecture/Power Supply/5V_K renamed /Project Architecture/Power Supply/12V_K
- net /Project Architecture/Power Supply/LDO_CD renamed /Project Architecture/Power Supply/LDO_CD_3v3
- net /Project Architecture/Power Supply/LDO_PWRGD renamed /Project Architecture/Power Supply/LDO_PWRGD_3v3
- net /Project Architecture/Power Supply/LDO_SENSE renamed /Project Architecture/Power Supply/LDO_SENSE_3v3
- net /Project Architecture/TRIAC/D3_K renamed /Project Architecture/TRIAC/D4_K
- net /Project Architecture/TRIAC/D_R5_OPTO renamed /Project Architecture/TRIAC/D_R5_OPTO_TOP
- net /Project Architecture/TRIAC/L1_F2 renamed /Project Architecture/TRIAC/L1_F2_TOP
- net /Project Architecture/TRIAC/L1_F2_OPTO renamed /Project Architecture/TRIAC/L1_F2_OPTO_TOP
- net /Project Architecture/TRIAC/L1_F2_RC renamed /Project Architecture/TRIAC/L1_F2_RC_TOP
- net /Project Architecture/TRIAC/L1_HEATER renamed /Project Architecture/TRIAC/L1_TOP
- net /Project Architecture/TRIAC/LN_OPTO renamed /Project Architecture/TRIAC/LN_OPTO_TOP
- C3 pad 1: /Project Architecture/Power Supply/LDO_VOUT -> +3.3V
- C4 pad 1: +5V -> +12V
- C5 pad 1: +5V -> +12V
- C6 pad 1: +5V -> +12V
- D2 pad 2: +5V -> +12V
- D6 pad 1: +5V -> +12V
- D7 pad 1: +5V -> +12V
- D8 pad 1: +5V -> +12V
- J2 pad 1: +3.3V -> /Project Architecture/TRIAC/L1_BOT
- J2 pad 2: GND -> GNDPWR
- J3 pad 1: +5V -> /Project Architecture/Thermocouple/TC_P
- J3 pad 2: GND -> /Project Architecture/Thermocouple/TC_N
- J6 pad 1: +5V -> +12V
- J7 pad 1: +5V -> +12V
- JP1 pad 1: /Project Architecture/Power Supply/LDO_VOUT -> /Project Architecture/Power Supply/LDO_VOUT_3v3
- JP2 pad 2: +5V -> +12V
- NT1 pad 2: /Project Architecture/Power Supply/LDO_VOUT -> /Project Architecture/Power Supply/LDO_VOUT_3v3
- R1 pad 1: /Project Architecture/Power Supply/LDO_VOUT -> /Project Architecture/Power Supply/LDO_VOUT_3v3
- R9 pad 2: D_Heater -> Top_Heater
- U1 pad 8: /Project Architecture/Power Supply/LDO_VOUT -> /Project Architecture/Power Supply/LDO_VOUT_3v3
- U4 pad 2: D_Heater -> Top_Heater
Other:
- board outline added: 229.8 x 182 mm

Commit message: work on pcb design
Parts:
- removed the ? at (317.5, 117.0)
- removed the ? at (541.5, 117.2)
- removed the ? at (317.5, 38.0)
- removed the C7 at (128.4, 101.6)
- added L1: 2.2uH, Inductor_SMD:L_1008_2520Metric_Pad1.43x2.20mm_HandSolder, F.Cu at (391.1, 122.2)
- moved R50 303.9 mm to (396.8, 156.2), turned to 180 degrees
- moved R49 297.6 mm to (390.3, 154.7), turned to -90 degrees
- moved C32 294.2 mm to (393.3, 154.7), turned to -90 degrees
- moved D11 292.8 mm to (396.8, 153.2), turned to 180 degrees
- moved NT2 289.4 mm to (387.8, 153.0), turned to 90 degrees
- moved JP8 288.3 mm to (392.0, 149.2), turned to 90 degrees
- moved TP17 287.4 mm to (378.3, 159.2), turned to -90 degrees
- moved C31 286.3 mm to (384.3, 158.2), turned to 180 degrees
- moved U12 286.1 mm to (385.3, 154.2)
- moved C7 281.6 mm to (385.5, 130.9), turned to 90 degrees
- moved C30 281.5 mm to (379.8, 152.7), turned to -90 degrees
- moved TP18 280.3 mm to (372.2, 159.2), turned to -90 degrees
- moved R52 279.9 mm to (397.6, 127.2)
- moved C34 279.0 mm to (385.6, 122.7), turned to -90 degrees
- moved F1 278.1 mm to (405.5, 89.2), turned to 180 degrees
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Other:
- board size 229.8 x 182 mm -> 225.8 x 224.2 mm

Commit message: working on pcb layout after bringing in work from laptop
Parts:
- removed ? (x3): , 
- removed FB1: WLBD2012HCU601TH, Inductor_SMD:L_0805_2012Metric_Pad1.05x1.20mm_HandSolder
- removed J14: Conn_01x06, Connector_PinHeader_2.54mm:PinHeader_1x06_P2.54mm_Vertical
- removed TP17, TP18: TestPoint, TestPoint:TestPoint_Pad_4.0x4.0mm
- removed U5: DS18B20+, Package_TO_SOT_THT:TO-92_Inline
- added C36: 100nF, Capacitor_SMD:C_0805_2012Metric_Pad1.18x1.45mm_HandSolder, F.Cu at (305.1, 44.7)
- added C37: 100nF, Capacitor_SMD:C_0805_2012Metric_Pad1.18x1.45mm_HandSolder, F.Cu at (305.1, 41.7)
- added C38: 10uF, Capacitor_SMD:C_0603_1608Metric_Pad1.08x0.95mm_HandSolder, F.Cu at (326.9, 44.5)
- added D14: RED, LED_SMD:LED_0603_1608Metric_Pad1.05x0.95mm_HandSolder, F.Cu at (191.8, 131.2)
- added D15: RED, LED_SMD:LED_0603_1608Metric_Pad1.05x0.95mm_HandSolder, F.Cu at (39.0, 106.0)
- added J12: Conn_01x04, Connector_JST:JST_XH_B4B-XH-A_1x04_P2.50mm_Vertical, F.Cu at (202.0, 85.2)
- added NT3: NetTie_2, NetTie:NetTie-2_SMD_Pad0.5mm, F.Cu at (218.5, 119.1)
- added NT4: NetTie_2, NetTie:NetTie-2_SMD_Pad0.5mm, F.Cu at (218.9, 112.6)
- added Q7: IRLML6244TRPBF, Package_TO_SOT_SMD:SOT-23, F.Cu at (40.5, 99.5)
- added R56: 1k, Resistor_SMD:R_0603_1608Metric_Pad0.98x0.95mm_HandSolder, F.Cu at (40.8, 103.0)
- added R57: 10k, Resistor_SMD:R_0603_1608Metric_Pad0.98x0.95mm_HandSolder, F.Cu at (37.0, 103.0)
- added R58: 220, Resistor_SMD:R_0603_1608Metric_Pad0.98x0.95mm_HandSolder, F.Cu at (188.0, 131.2)
- added R59: 1k, Resistor_SMD:R_0603_1608Metric_Pad0.98x0.95mm_HandSolder, F.Cu at (37.5, 99.5)
- added TP7: TestPoint, TestPoint:TestPoint_Keystone_5019_Miniature, F.Cu at (229.0, 48.0)
- added TP8: TestPoint, TestPoint:TestPoint_Keystone_5019_Miniature, F.Cu at (319.6, 24.4)
- added U14: DS18B20+, Connector_JST:JST_XH_B3B-XH-A_1x03_P2.50mm_Vertical, F.Cu at (162.8, 115.8)
- added U15: DS18B20+, Connector_JST:JST_XH_B3B-XH-A_1x03_P2.50mm_Vertical, F.Cu at (179.0, 115.8)
- C10: value 20pF -> 22uF; footprint Capacitor_SMD:C_0402_1005Metric_Pad0.74x0.62mm_HandSolder -> Capacitor_SMD:C_1206_3216Metric_Pad1.33x1.80mm_HandSolder
- C11: value 100nF -> 1uF; footprint Capacitor_SMD:C_0603_1608Metric_Pad1.08x0.95mm_HandSolder -> Capacitor_SMD:C_0805_2012Metric_Pad1.18x1.45mm_HandSolder
- C12: value 2.2uF Low ESR -> 100nF; footprint Capacitor_SMD:C_0805_2012Metric_Pad1.18x1.45mm_HandSolder -> Capacitor_SMD:C_0603_1608Metric_Pad1.08x0.95mm_HandSolder
- C13: value 1uF -> 10uF
- C15, C16: value 100nF -> 20pF; footprint Capacitor_SMD:C_0603_1608Metric_Pad1.08x0.95mm_HandSolder -> Capacitor_SMD:C_0402_1005Metric_Pad0.74x0.62mm_HandSolder
- C18: value 100nF -> 2.2uF Low ESR; footprint Capacitor_SMD:C_0603_1608Metric_Pad1.08x0.95mm_HandSolder -> Capacitor_SMD:C_0805_2012Metric_Pad1.18x1.45mm_HandSolder
- C19: value 10nF 250V -> 1uF; footprint Capacitor_SMD:C_1812_4532Metric_Pad1.57x3.40mm_HandSolder -> Capacitor_SMD:C_0805_2012Metric_Pad1.18x1.45mm_HandSolder
- C20, C24: value 1uF X7R -> 100nF
- C21, C22: footprint Capacitor_SMD:C_0805_2012Metric_Pad1.18x1.45mm_HandSolder -> Capacitor_SMD:C_0603_1608Metric_Pad1.08x0.95mm_HandSolder
- C23: value 10nF 250V -> 100nF; footprint Capacitor_SMD:C_1812_4532Metric_Pad1.57x3.40mm_HandSolder -> Capacitor_SMD:C_0603_1608Metric_Pad1.08x0.95mm_HandSolder
- C25, C26: value 100nF -> 10nF 250V; footprint Capacitor_SMD:C_0805_2012Metric_Pad1.18x1.45mm_HandSolder -> Capacitor_SMD:C_1812_4532Metric_Pad1.57x3.40mm_HandSolder
- C28: value 100nF -> 1uF X7R; footprint Capacitor_SMD:C_0805_2012Metric_Pad1.18x1.45mm_HandSolder -> Capacitor_SMD:C_0603_1608Metric_Pad1.08x0.95mm_HandSolder
- C3: footprint Capacitor_SMD:C_0805_2012Metric_Pad1.18x1.45mm_HandSolder -> KemetA765:CAPAE830X730N
- C30, C32: value 10uF -> 100nF
- C31: value 1uF -> 100nF
- C33: value 100nF -> 10uF
- C34: value 22uF -> 10uF; footprint Capacitor_THT:C_Radial_D5.0mm_H11.0mm_P2.00mm -> Capacitor_SMD:C_0603_1608Metric_Pad1.08x0.95mm_HandSolder
- C35: value 22uF -> 1uF X7R; footprint Capacitor_THT:C_Radial_D5.0mm_H11.0mm_P2.00mm -> Capacitor_SMD:C_0603_1608Metric_Pad1.08x0.95mm_HandSolder
- C4: value 47uF -> 10uF; footprint Capacitor_THT:C_Radial_D5.0mm_H11.0mm_P2.00mm -> Capacitor_SMD:C_0805_2012Metric_Pad1.18x1.45mm_HandSolder
- C5: value 1uF -> 100nF; footprint Capacitor_SMD:C_0805_2012Metric_Pad1.18x1.45mm_HandSolder -> Capacitor_SMD:C_0603_1608Metric_Pad1.08x0.95mm_HandSolder
- C6: value 100nF -> 10uF; footprint Capacitor_SMD:C_0603_1608Metric_Pad1.08x0.95mm_HandSolder -> Capacitor_SMD:C_0805_2012Metric_Pad1.18x1.45mm_HandSolder
- C7: value 10uF -> 1uF; footprint Capacitor_THT:C_Radial_D5.0mm_H11.0mm_P2.00mm -> Capacitor_SMD:C_0805_2012Metric_Pad1.18x1.45mm_HandSolder
- C8: value 100nF -> 22uF; footprint Capacitor_SMD:C_0603_1608Metric_Pad1.08x0.95mm_HandSolder -> Capacitor_SMD:C_1206_3216Metric_Pad1.33x1.80mm_HandSolder
- C9: value 20pF -> 47uF; footprint Capacitor_SMD:C_0402_1005Metric_Pad0.74x0.62mm_HandSolder -> Capacitor_SMD:C_Elec_6.3x5.8
- D10: value T2035T-8G-RT -> 1N5819HW-7-F; footprint Package_TO_SOT_THT:TO-220-3_Vertical -> Diode_SMD:D_SOD-123
- D11, D12: value RED -> 1N5819HW-7-F; footprint LED_SMD:LED_0603_1608Metric_Pad1.05x0.95mm_HandSolder -> Diode_SMD:D_SOD-123
- D5: value T2035T-8G-RT -> GRN; footprint Package_TO_SOT_THT:TO-220-3_Vertical -> LED_SMD:LED_0603_1608Metric_Pad1.05x0.95mm_HandSolder
- D6, D7: value 1N5819HW-7-F -> T2035T-8G-RT; footprint Diode_SMD:D_SOD-123 -> Package_TO_SOT_THT:TO-220-3_Vertical
- D8: value 1N5819HW-7-F -> RED; footprint Diode_SMD:D_SOD-123 -> LED_SMD:LED_0603_1608Metric_Pad1.05x0.95mm_HandSolder
- J10: value Conn_01x04 -> Conn_01x06; footprint Connector_JST:JST_XH_B4B-XH-A_1x04_P2.50mm_Vertical -> Connector_PinHeader_2.54mm:PinHeader_1x06_P2.54mm_Vertical
- J11: value Conn_01x04 -> Conn_01x07; footprint Connector_JST:JST_XH_B4B-XH-A_1x04_P2.50mm_Vertical -> Connector_JST:JST_XH_B7B-XH-A_1x07_P2.50mm_Vertical
- J13: value Conn_02x05_Odd_Even -> Conn_01x04; footprint Connector_IDC:IDC-Header_2x05_P2.54mm_Vertical -> Connector_JST:JST_XH_B4B-XH-A_1x04_P2.50mm_Vertical
- J15: value Conn_01x08 -> Conn_02x05_Odd_Even; footprint Connector_PinHeader_2.54mm:PinHeader_1x08_P2.54mm_Vertical -> Connector_IDC:IDC-Header_2x05_P2.54mm_Vertical
- J16: value 4DB-P108-02 -> Conn_01x02; footprint 4DB_P108_02:CONN_4DB-P108-02_TEC -> TerminalBlock_Phoenix:TerminalBlock_Phoenix_MKDS-1,5-2-5.08_1x02_P5.08mm_Horizontal
- J17: value Conn_01x02 -> Conn_01x06; footprint TerminalBlock_Phoenix:TerminalBlock_Phoenix_MKDS-1,5-2-5.08_1x02_P5.08mm_Horizontal -> Connector_PinHeader_2.54mm:PinHeader_1x06_P2.54mm_Vertical
- J3: value 4DB-P108-02 -> 1366005; footprint 4DB_P108_02:CONN_4DB-P108-02_TEC -> PhoenixContact_SPTA:SPTA-THR 2.53-5.0 P26
- J4: value 1366005 -> 4DB-P108-02; footprint PhoenixContact_SPTA:SPTA-THR 2.53-5.0 P26 -> 4DB_P108_02:CONN_4DB-P108-02_TEC
- J6: value Conn_01x02 -> 4DB-P108-02; footprint Connector_JST:JST_XH_B2B-XH-A_1x02_P2.50mm_Vertical -> 4DB_P108_02:CONN_4DB-P108-02_TEC
- J9: value Conn_01x07 -> Conn_01x02; footprint Connector_JST:JST_XH_B7B-XH-A_1x07_P2.50mm_Vertical -> Connector_JST:JST_XH_B2B-XH-A_1x02_P2.50mm_Vertical
- JP3, JP4: footprint Jumper:SolderJumper-2_P1.3mm_Open_TrianglePad1.0x1.5mm -> Connector_PinHeader_2.54mm:PinHeader_1x02_P2.54mm_Vertical
- JP8, JP9: footprint Connector_PinHeader_2.54mm:PinHeader_1x02_P2.54mm_Vertical -> Jumper:SolderJumper-2_P1.3mm_Open_TrianglePad1.0x1.5mm
- R10, R53, R9: value 330 -> 10k
- R11: value 330 -> 220; footprint Resistor_SMD:R_2512_6332Metric_Pad1.40x3.35mm_HandSolder -> Resistor_SMD:R_0603_1608Metric_Pad0.98x0.95mm_HandSolder
- R12: value 330 -> 39
- R14, R15: value 100k -> 330; footprint Resistor_SMD:R_0603_1608Metric_Pad0.98x0.95mm_HandSolder -> Resistor_SMD:R_2512_6332Metric_Pad1.40x3.35mm_HandSolder
- R16: value 560 -> 330; footprint Resistor_SMD:R_0603_1608Metric_Pad0.98x0.95mm_HandSolder -> Resistor_SMD:R_2512_6332Metric_Pad1.40x3.35mm_HandSolder
- R17: value TC33X-2-102E -> 330; footprint Potentiometer_SMD:Potentiometer_Bourns_TC33X_Vertical -> Resistor_SMD:R_2512_6332Metric_Pad1.40x3.35mm_HandSolder
- R18: value 280k -> 220
- R19: value TC33X-2-104E -> 220; footprint Potentiometer_SMD:Potentiometer_Bourns_TC33X_Vertical -> Resistor_SMD:R_0603_1608Metric_Pad0.98x0.95mm_HandSolder
- R20, R21: value 1k -> 330
- R22, R23, R54: value 1k -> 10k
- R24, R6: value 220 -> 330
- R25: value 10k -> 330
- R26, R27, R28: value 10k -> 100k
- R29, R41: value 1k -> 100k
- R3: value 1.2k -> 52.3k
- R30: value 330 -> 560
- R31: value 330 -> TC33X-2-102E; footprint Resistor_SMD:R_0603_1608Metric_Pad0.98x0.95mm_HandSolder -> Potentiometer_SMD:Potentiometer_Bourns_TC33X_Vertical
- R32: value 330 -> 560; footprint Resistor_SMD:R_2512_6332Metric_Pad1.40x3.35mm_HandSolder -> Resistor_SMD:R_0603_1608Metric_Pad0.98x0.95mm_HandSolder
- R33: value 330 -> TC33X-2-102E; footprint Resistor_SMD:R_2512_6332Metric_Pad1.40x3.35mm_HandSolder -> Potentiometer_SMD:Potentiometer_Bourns_TC33X_Vertical
- R34: value 39 -> 280k; footprint Resistor_SMD:R_2512_6332Metric_Pad1.40x3.35mm_HandSolder -> Resistor_SMD:R_0603_1608Metric_Pad0.98x0.95mm_HandSolder
- R35: value 100k -> 280k
- R36: value 100k -> TC33X-2-104E; footprint Resistor_SMD:R_0603_1608Metric_Pad0.98x0.95mm_HandSolder -> Potentiometer_SMD:Potentiometer_Bourns_TC33X_Vertical
- R37: value 560 -> TC33X-2-104E; footprint Resistor_SMD:R_0603_1608Metric_Pad0.98x0.95mm_HandSolder -> Potentiometer_SMD:Potentiometer_Bourns_TC33X_Vertical
- R38: value TC33X-2-102E -> 1k; footprint Potentiometer_SMD:Potentiometer_Bourns_TC33X_Vertical -> Resistor_SMD:R_0603_1608Metric_Pad0.98x0.95mm_HandSolder
- R39, R46: value 280k -> 1k
- R40: value TC33X-2-104E -> 100k; footprint Potentiometer_SMD:Potentiometer_Bourns_TC33X_Vertical -> Resistor_SMD:R_0603_1608Metric_Pad0.98x0.95mm_HandSolder
- R42: value 100k -> 560
- R43: value 100k -> TC33X-2-102E; footprint Resistor_SMD:R_0603_1608Metric_Pad0.98x0.95mm_HandSolder -> Potentiometer_SMD:Potentiometer_Bourns_TC33X_Vertical
- R44: value 560 -> 280k
- R45: value TC33X-2-102E -> TC33X-2-104E
- R47: value TC33X-2-104E -> 1k; footprint Potentiometer_SMD:Potentiometer_Bourns_TC33X_Vertical -> Resistor_SMD:R_0603_1608Metric_Pad0.98x0.95mm_HandSolder
- R49, R55: value 10k -> 1k
- R51: value 52.3k -> 10k
- R7: value 10k -> 1.2k
- TP1, TP2, TP3, TP4: footprint TestPoint:TestPoint_Keystone_5019_Miniature -> TestPoint:TestPoint_Pad_4.0x4.0mm
- TP5, TP6: footprint TestPoint:TestPoint_Pad_4.0x4.0mm -> TestPoint:TestPoint_Keystone_5019_Miniature
- U10: value OPA333AIDCKT -> DS18B20+; footprint Package_SO:SOIC-8_3.9x4.9mm_P1.27mm -> Package_TO_SOT_THT:TO-92_Inline
- U12: value MCP1727T-3302E/SN -> OPA333AIDCKT
- U13: value AP62250WU -> DS18B20+; footprint Package_TO_SOT_SMD:TSOT-23-6_HandSoldering -> Package_TO_SOT_THT:TO-92_Inline
- U2: value STM32F401RETx -> AP62250WU; footprint Package_QFP:LQFP-64_10x10mm_P0.5mm -> Package_TO_SOT_SMD:TSOT-23-6_HandSoldering
- U3: value DS18B20+ -> MCP1727T-3302E/SN; footprint Package_TO_SOT_THT:TO-92_Inline -> Package_SO:SOIC-8_3.9x4.9mm_P1.27mm
- U4: value MOC3083S-TA1 -> STM32F401RETx; footprint Package_DIP:SMDIP-6_W9.53mm -> Package_QFP:LQFP-64_10x10mm_P0.5mm
- U6: value OPA333AIDCKT -> MOC3083S-TA1; footprint Package_SO:SOIC-8_3.9x4.9mm_P1.27mm -> Package_DIP:SMDIP-6_W9.53mm
- U9: value DS18B20+ -> OPA333AIDCKT; footprint Package_TO_SOT_THT:TO-92_Inline -> Package_SO:SOIC-8_3.9x4.9mm_P1.27mm
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Connections:
- net Net-(F4-Pad1) renamed /Project Architecture/Peripherals and Connectors/CONVFAN_L1_FUSED
- C10 pad 1: /Project Architecture/MCU/HSE_OUT -> /Project Architecture/Power Supply/5V_BUCK_VOUT
- C11 pad 1: GND -> +12V
- C11 pad 2: NRST_SW -> GND
- C12 pad 1: /Project Architecture/MCU/STM_VCAP -> +12V
- C13 pad 1: +3.3V -> +3.3VA
- C14 pad 1: +3.3V -> +3.3VA
- C15 pad 1: +3.3V -> /Project Architecture/MCU/HSE_IN
- C15 pad 2: GND -> /Project Architecture/MCU/HSE_GND
- C16 pad 1: +3.3V -> /Project Architecture/MCU/HSE_OUT
- C16 pad 2: GND -> /Project Architecture/MCU/HSE_GND
- C17 pad 1: +3.3V -> GND
- C17 pad 2: GND -> NRST_SW
- C18 pad 1: +3.3V -> /Project Architecture/MCU/STM_VCAP
- C19 pad 1: /Project Architecture/TRIAC/L1_F2_RC_TOP -> +3.3V
- C19 pad 2: LN -> GND
- C20 pad 1: /Project Architecture/Thermocouple/TC_NON -> +3.3V
- C21 pad 1: /Project Architecture/Thermocouple/TC_INV -> +3.3V
- C21 pad 2: /Project Architecture/Thermocouple/TC_S1_OUT -> GND
- C22 pad 1: +3.3VA -> +3.3V
- C23 pad 1: /Project Architecture/TRIAC/L1_F2_RC_BOT -> +3.3V
- C23 pad 2: LN -> GND
- C24 pad 1: /Project Architecture/Thermocouple/TC_NON -> +3.3V
- C25 pad 1: /Project Architecture/Thermocouple/TC_INV -> /Project Architecture/TRIAC/L1_F2_RC_TOP
- C25 pad 2: /Project Architecture/Thermocouple/TC_S1_OUT -> LN
- C26 pad 1: +3.3VA -> /Project Architecture/TRIAC/L1_F2_RC_BOT
- C26 pad 2: GND -> LN
- C27 pad 1: /Project Architecture/Thermocouple/TC_NON -> /Project Architecture/Thermocouple/TC1_AFE_NON
- C28 pad 1: /Project Architecture/Thermocouple/TC_INV -> /Project Architecture/Thermocouple/TC2_AFE_NON
- C28 pad 2: /Project Architecture/Thermocouple/TC_S1_OUT -> GND
- C29 pad 1: +3.3VA -> /Project Architecture/Thermocouple/TC1_AFE_INV
- C29 pad 2: GND -> /Project Architecture/Thermocouple/TC1_AFE_OUT
- C3 pad 1: +3.3V -> +12V
- C30 pad 1: +5V -> /Project Architecture/Thermocouple/TC2_AFE_INV
- C30 pad 2: GND -> /Project Architecture/Thermocouple/TC2_AFE_OUT
- C31 pad 1: /Project Architecture/Power Supply/LDO_CD_3v3A -> +3.3VA
- C33 pad 1: Net-(U13-SW) -> TC1_ADC
- C33 pad 2: Net-(U13-BST) -> GND
- C34 pad 1: +5V -> TC2_ADC
- C35 pad 1: +5V -> /Project Architecture/Thermocouple/TC3_AFE_NON
- C4 pad 1: +12V -> +3.3V
- C5 pad 1: +12V -> /Project Architecture/Power Supply/5V_BUCK_SW
- C5 pad 2: GND -> /Project Architecture/Power Supply/5V_BUCK_BST
- C6 pad 1: +12V -> +5V
- C7 pad 1: +12V -> /Project Architecture/Power Supply/LDO_CD_3v3A
- C8 pad 1: +3.3VA -> /Project Architecture/Power Supply/5V_BUCK_VOUT
- C9 pad 1: /Project Architecture/MCU/HSE_IN -> +12V
- D10 pad 1: LN -> +12V
- D10 pad 2: /Project Architecture/TRIAC/L1_F2_BOT -> /Project Architecture/Peripherals and Connectors/FAN1_MINUS
- D11 pad 1: /Project Architecture/Power Supply/3V3A_K -> +12V
- D11 pad 2: +3.3VA -> /Project Architecture/Peripherals and Connectors/FAN2_MINUS
- D12 pad 1: Net-(D12-K) -> +12V
- D12 pad 2: +5V -> /Project Architecture/Peripherals and Connectors/FAN3_MINUS
- D13 pad 2: /Project Architecture/Peripherals and Connectors/FAN3_MINUS -> /Project Architecture/Peripherals and Connectors/CONVFAN_RELAY_MINUS
- D2 pad 1: /Project Architecture/Power Supply/12V_K -> /Project Architecture/Power Supply/5V_K
- D2 pad 2: +12V -> +5V
- D3 pad 1: /Project Architecture/MCU/STM_USR_LED_K -> /Project Architecture/Power Supply/12V_K
- D3 pad 2: /Project Architecture/MCU/STM_USR_LED -> +12V
- D4 pad 1: /Project Architecture/TRIAC/D4_K -> /Project Architecture/Power Supply/3V3A_K
- D4 pad 2: +5V -> +3.3VA
- D5 pad 1: LN -> /Project Architecture/MCU/STM_USR_LED1_K
- D5 pad 2: /Project Architecture/TRIAC/L1_F2_TOP -> /Project Architecture/MCU/STM_USR_LED1
- D6 pad 1: +12V -> LN
- D6 pad 2: /Project Architecture/Peripherals and Connectors/FAN1_MINUS -> /Project Architecture/TRIAC/L1_F2_TOP
- D7 pad 1: +12V -> LN
- D7 pad 2: /Project Architecture/Peripherals and Connectors/FAN2_MINUS -> /Project Architecture/TRIAC/L1_F2_BOT
- D8 pad 1: +12V -> /Project Architecture/TRIAC/D4_K
- D8 pad 2: /Project Architecture/Peripherals and Connectors/FAN3_MINUS -> +5V
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Routing:
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- added copper zone on F.Cu, net /Project Architecture/TRIAC/L1_BOT
- added copper zone on F.Cu, net /Project Architecture/TRIAC/L1_F2_BOT
- added copper zone on F.Cu, net /Project Architecture/TRIAC/L1_F2_TOP
- added copper zone on F.Cu, net /Project Architecture/TRIAC/L1_TOP
- added copper zone on F.Cu, net L1
- added copper zone on F.Cu, net LN
Other:
- board size 225.8 x 224.2 mm -> 221.8 x 159.2 mm
- board text added: "+"
- board text added: "+ -"
- board text added: "+12V"
- board text added: "+3v3"
- board text added: "+3v3A"
- board text added: "+5V"
- board text added: "+5v"
- board text added: "-"
- board text added: "12V Enable"
- board text added: "12V Fan 2"
- board text added: "12V Fan 3"
- board text added: "3V3 Enable"
- board text added: "3V3A Enable"
- board text added: "3v3"
- board text added: "5V Enable"
- board text added: "BOOT0"
- board text added: "BOTTOM"
- board text added: "Bootloader"
- board text added: "Bottom"
- board text added: "Button Header"
- board text added: "Data"
- board text added: "Error"
- board text added: "Feedback"
- board text added: "GND"
- board text added: "GPIO"
- board text added: "I2C OLED"
- board text added: "Keypad Matrix"
- board text added: "Normal"
- board text added: "Oven Fan"
- board text added: "PD"
- board text added: "PWR"
- board text added: "RST"
- board text added: "Reset"
- board text added: "STLink Power"
- board text added: "STLink Programmer"
- board text added: "Status"
- board text added: "TOP"
- board text added: "TRIAC Heatsink Fan 12V"
- board text added: "Top"
- board text added: "Vout"
