File: mainBoard/mainBoard.kicad_pcb (KiCad board)
At the start: 4 copper layers, 221.8 x 159.2 mm, 199 parts, among them J1 1366005, J10 Conn_01x06, J11 Conn_01x07, J12 Conn_01x04, J13 Conn_01x04, J15 Conn_02x05_Odd_Even, J16 Conn_01x02, J17 Conn_01x06, J2 1366005, J3 1366005, J4 4DB-P108-02, J5 4DB-P108-02, J6 4DB-P108-02, J7 Conn_01x02, J8 Conn_01x02, J9 Conn_01x02, K1 Relay_SPDT, Q1 IRLML6244TRPBF, Q2 IRLML6244TRPBF, Q3 IRLML6244TRPBF, Q4 IRLML6244TRPBF, Q5 IRLML6244TRPBF, Q6 IRLML6244TRPBF, Q7 IRLML6244TRPBF, SW1 SW_SPST, SW2 SW_SPDT, SW3 SW_Push, U1 MCP1727T-3302E/SN, U10 DS18B20+, U11 DS18B20+, U12 OPA333AIDCKT, U13 DS18B20+, U14 DS18B20+, U15 DS18B20+, U2 AP62250WU, U3 MCP1727T-3302E/SN, U4 STM32F401RETx, U6 MOC3083S-TA1, U7 MOC3083S-TA1, U8 OPA333AIDCKT, U9 OPA333AIDCKT, Y1 ATS240C-E

Commit message: board routing nearly complete
Parts:
- added G***: LOGO, LOGO, F.Cu at (-19.1, 67.7)
- added G***: LOGO, LOGO, F.Cu at (142.8, 48.5)
- added REF**: MTP Logo 5mm Low Detail, Watermarks:MTP Logo 5mm Low Detail, F.Cu at (157.8, 132.2)
- J17: value Conn_01x06 -> Conn_01x05; footprint Connector_PinHeader_2.54mm:PinHeader_1x06_P2.54mm_Vertical -> Connector_PinHeader_2.54mm:PinHeader_1x05_P2.54mm_Vertical
- moved R43 133.9 mm to (210.9, 93.9), turned to -90 degrees
- moved R45 132.3 mm to (215.9, 95.4), turned to -90 degrees
- moved U13 130.8 mm to (208.5, 78.8), turned to 90 degrees
- moved R39 128.1 mm to (213.0, 106.0), turned to -90 degrees
- moved JP7 126.7 mm to (229.6, 94.2), turned to -90 degrees
- moved C38 126.2 mm to (220.2, 112.0), turned to 0 degrees
- moved C34 125.1 mm to (215.8, 107.0), turned to 0 degrees
- moved TP15 120.8 mm to (206.9, 94.2), turned to -90 degrees
- moved R46 118.5 mm to (220.2, 113.8)
- moved TP14 115.3 mm to (206.9, 87.4), turned to -90 degrees
- moved R42 113.3 mm to (211.1, 89.2)
- moved JP6 109.8 mm to (234.8, 73.5), turned to -90 degrees
- moved R44 109.1 mm to (216.9, 90.2), turned to -90 degrees
- moved C35 108.0 mm to (226.1, 86.0), turned to 0 degrees
- moved R41 107.8 mm to (215.1, 86.2), turned to 0 degrees
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Connections:
- C34 pad 1: TC2_ADC -> TC3_ADC
- C38 pad 1: TC3_ADC -> TC2_ADC
- J17 pad 1: unconnected-(J17-Pin_1-Pad1) -> PB12
- J17 pad 2: PC8 -> PB13
- J17 pad 3: PC9 -> PB14
- J17 pad 4: PB2 -> PB15
- J17 pad 5: PB1 -> PC6
- J5 pad 1: /Project Architecture/Thermocouple/TC2_P -> /Project Architecture/Thermocouple/TC2_N
- J5 pad 2: /Project Architecture/Thermocouple/TC2_N -> /Project Architecture/Thermocouple/TC2_P
- J6 pad 1: /Project Architecture/Thermocouple/TC3_P -> /Project Architecture/Thermocouple/TC3_N
- J6 pad 2: /Project Architecture/Thermocouple/TC3_N -> /Project Architecture/Thermocouple/TC3_P
- R39 pad 1: /Project Architecture/Thermocouple/TC2_ADC_RC -> /Project Architecture/Thermocouple/TC3_ADC_RC
- R39 pad 2: TC2_ADC -> TC3_ADC
- R46 pad 1: /Project Architecture/Thermocouple/TC3_ADC_RC -> /Project Architecture/Thermocouple/TC2_ADC_RC
- R46 pad 2: TC3_ADC -> TC2_ADC
- U4 pad 15: unconnected-(U4-PA1-Pad15) -> Soft_Power
- U4 pad 16: TC3_ADC -> TC2_ADC
- U4 pad 17: unconnected-(U4-PA3-Pad17) -> TC2_CJ_TEMP
- U4 pad 20: TC2_ADC -> TC3_ADC
- U4 pad 21: TC1_ADC -> unconnected-(U4-PA5-Pad21)
- U4 pad 23: TC2_CJ_TEMP -> TC1_ADC
- U4 pad 25: Soft_Power -> unconnected-(U4-PC5-Pad25)
- U4 pad 26: PB0 -> unconnected-(U4-PB0-Pad26)
- U4 pad 27: PB1 -> unconnected-(U4-PB1-Pad27)
- U4 pad 28: PB2 -> unconnected-(U4-PB2-Pad28)
- U4 pad 33: unconnected-(U4-PB12-Pad33) -> PB12
- U4 pad 34: unconnected-(U4-PB13-Pad34) -> PB13
- U4 pad 35: unconnected-(U4-PB14-Pad35) -> PB14
- U4 pad 36: unconnected-(U4-PB15-Pad36) -> PB15
- U4 pad 37: unconnected-(U4-PC6-Pad37) -> PC6
- U4 pad 43: Fan2 -> Fan1
- U4 pad 44: Fan3 -> Fan2
- U4 pad 45: Fan1 -> Fan3
Routing:
- net +5V: track 0.00 -> 263.0 mm, vias 0 -> 4
- net +12V: track 0.00 -> 252.7 mm
- net Conv_Fan: track 0.00 -> 194.5 mm, vias 0 -> 4
- net GND: track 0.00 -> 175.7 mm, vias 0 -> 96
- net Fan1: track 0.00 -> 174.5 mm, vias 0 -> 4
- net +3.3VA: track 0.00 -> 133.1 mm, vias 0 -> 7
- net Fan2: track 0.00 -> 87.5 mm, vias 0 -> 2
- net Fan3: track 0.00 -> 84.2 mm, vias 0 -> 2
- net TC2_CJ_TEMP: track 0.00 -> 82.3 mm
- net TC1_CJ_TEMP: track 0.00 -> 81.4 mm
- net NRST_SW: track 0.00 -> 68.7 mm
- net TRIAC_TOP_TEMP: track 0.00 -> 47.0 mm
- net /Project Architecture/Thermocouple/TC2_ADC_RC: track 0.00 -> 46.8 mm
- net Top_Heater: track 0.00 -> 45.8 mm
- net SWDIO: track 0.00 -> 45.6 mm, vias 0 -> 2
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- added copper zone on F.Cu, net +3.3V
- added copper zone on In2.Cu, net +3.3V
- added copper zone on F.Cu, net /Project Architecture/Peripherals and Connectors/STLink_+3v3
- added copper zone on F.Cu, net /Project Architecture/Peripherals and Connectors/STLink_+5v
- added copper zone on F.Cu, net /Project Architecture/Power Supply/5V_BUCK_BST
- added copper zone on F.Cu, net /Project Architecture/Power Supply/5V_BUCK_SW
- added copper zone on F.Cu, net /Project Architecture/Power Supply/5V_BUCK_VOUT
- added copper zone on B.Cu, net GND
- added copper zone on F.Cu, net GND
Other:
- board size 221.8 x 159.2 mm -> 221.8 x 118.5 mm
- board text added: "10A Fuse"
- board text added: "12V Input"
- board text added: "1A Fuse"
- board text added: "3A Fuse"
- board text added: "5V"
- board text added: "AC Input"
- board text added: "Bottom Element"
- board text added: "C0 C1 C2 R0 R1 R2 R3"
- board text added: "CH 1"
- board text added: "CH 2"
- board text added: "CH 3"
- board text added: "L G N"
- board text added: "Michael Pate Version 3.0 06/2026"
- board text added: "N G L"
- board text added: "PB12"
- board text added: "PB13"
- board text added: "PB14"
- board text added: "PB15"
- board text added: "PC6"
- board text added: "Power Switch"
- board text added: "SCL"
- board text added: "SDA"
- board text added: "Toaster-Flo"
- board text added: "Top Element"
- board text removed: "BOTTOM"
- board text removed: "TOP"

Commit message: tweak board design more
Parts:
- added G***: LOGO, LOGO, F.Cu at (74.1, 85.9)
- added G***: LOGO, LOGO, F.Cu at (40.6, 42.4)
- added G***: LOGO, LOGO, B.Cu at (73.7, 80.8)
- added R60: 10k, Resistor_SMD:R_0603_1608Metric_Pad0.98x0.95mm_HandSolder, F.Cu at (229.8, 113.0)
- added REF**: MTP Logo 10mm Low Detail, Watermarks:MTP Logo 10mm Low Detail, F.Cu at (158.8, 50.2)
- added SW4: SW_Push, Button_Switch_THT:SW_PUSH_6mm_H4.3mm, F.Cu at (232.5, 114.0)
- moved G*** 207.4 mm to (172.9, -10.6)
- moved R10 6.47 mm to (243.6, 115.1), turned to 180 degrees
- moved C17 1.91 mm to (243.6, 113.4)
- moved G*** 0.25 mm to (142.8, 48.8)
Connections:
- U4 pad 14: unconnected-(U4-PA0-Pad14) -> /Project Architecture/MCU/STM_USR_BTN
Routing:
- net /Project Architecture/MCU/STM_USR_BTN: track 0.00 -> 30.8 mm, vias 0 -> 1
- net NRST_SW: track 68.7 -> 71.1 mm
- net +3.3V: track 44.6 -> 46.8 mm, vias 19 -> 20
- net /Project Architecture/Power Supply/L1_F1: track 16.5 -> 18.6 mm
- net SWDCLK: track 44.2 -> 45.4 mm
- net TC3_CJ_TEMP: track 45.1 -> 43.9 mm
- net GND: track 175.7 -> 175.1 mm
- added copper zone on In1.Cu, net GND
Other:
- outline, holes or cut-outs redrawn
- board text added: "120VAC"
- board text added: "120VAC Present on ALL HOT side terminals!"
- board text added: "COLD"
- board text added: "COLD Side"
- board text added: "HIGH VOLTAGE"
- board text added: "HOT"
- board text added: "HOT Side"
- board text added: "IN OUT"
- board text added: "User (PA0)"
