File: mainBoard/mcu.kicad_sch (KiCad schematic)
At the start: 23 parts, among them SW2 SW_SPDT, SW3 SW_Push, U4 STM32F401RETx, Y1 ATS240C-E

Commit message: board routing nearly complete
Connections:
- net Fan1: now also U4.43 (PA10); no longer U4.45 (PA12)
- net Fan2: now also U4.44 (PA11); no longer U4.43 (PA10)
- net Fan3: now also U4.45 (PA12); no longer U4.44 (PA11)
- net Soft_Power: now also U4.15 (PA1); no longer U4.25 (PC5)
- net TC1_ADC: now also U4.23 (PA7); no longer U4.21 (PA5)
- net TC2_ADC: now also U4.16 (PA2); no longer U4.20 (PA4)
- net TC2_CJ_TEMP: now also U4.17 (PA3); no longer U4.23 (PA7)
- net TC3_ADC: now also U4.20 (PA4); no longer U4.16 (PA2)
- net PB12: now reaches U4.33 (PB12)
- net PB13: now reaches U4.34 (PB13)
- net PB14: now reaches U4.35 (PB14)
- net PB15: now reaches U4.36 (PB15)
- net PC6: now reaches U4.37 (PC6)
- net PB0: no longer names the net of U4.26 (PB0)
- net PB1: no longer names the net of U4.27 (PB1)
- net PB2: no longer names the net of U4.28 (PB2)
- no-connect marks 16 -> 14
Changed lines of the file:
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@@
-	)
-	(no_connect
-		(at 234.95 189.23)
-	)
-	(no_connect
-		(at 237.49 196.85)
 	)
 	(no_connect
@@
 	)
 	(no_connect
-		(at 234.95 125.73)
-	)
-	(no_connect
 		(at 199.39 181.61)
 	)
@@
 	)
 	(no_connect
-		(at 234.95 186.69)
+		(at 199.39 184.15)
 	)
 	(no_connect
-		(at 199.39 184.15)
-	)
-	(no_connect
-		(at 199.39 161.29)
+		(at 237.49 163.83)
 	)
 	(no_connect
@@
 	)
 	(no_connect
-		(at 234.95 191.77)
+		(at 237.49 166.37)
 	)
 	(no_connect
-		(at 237.49 194.31)
+		(at 234.95 186.69)
+	)
+	(no_connect
+		(at 237.49 161.29)
 	)
 	(no_connect
@@
 	)
 	(no_connect
-		(at 234.95 120.65)
+		(at 199.39 158.75)
+	)
+	(no_connect
+		(at 234.95 130.81)
 	)
 	(wire
@@
 	(global_label "TC3_ADC"
 		(shape input)
-		(at 234.95 123.19 0)
-		(fields_autoplaced yes)
-		(effects
-			(font
-				(size 1.27 1.27)
-			)
-			(justify left)
-		)
-		(property "Intersheetrefs" "${INTERSHEET_REFS}"
-			(at 244.5481 123.19 0)
+		(at 234.95 128.27 0)
+		(fields_autoplaced yes)
+		(effects
+			(font
+				(size 1.27 1.27)
+			)
+			(justify left)
+		)
+		(property "Intersheetrefs" "${INTERSHEET_REFS}"
+			(at 244.5481 128.27 0)
 			(hide yes)
 			(show_name no)
@@
 	(global_label "Soft_Power"
 		(shape input)
-		(at 199.39 158.75 180)
-		(fields_autoplaced yes)
-		(effects
-			(font
-				(size 1.27 1.27)
-			)
-			(justify right)
-		)
-		(property "Intersheetrefs" "${INTERSHEET_REFS}"
-			(at 186.8625 158.75 0)
-			(hide yes)
-			(show_name no)
-			(do_not_autoplace no)
-			(effects
-				(font
-					(size 1.27 1.27)
-				)
-				(justify right)
+		(at 234.95 120.65 0)
+		(fields_autoplaced yes)
+		(effects
+			(font
+				(size 1.27 1.27)
+			)
+			(justify left)
+		)
+		(property "Intersheetrefs" "${INTERSHEET_REFS}"
+			(at 248.337 120.65 0)
+			(hide yes)
+			(show_name no)
+			(do_not_autoplace no)
+			(effects
+				(font
+					(size 1.27 1.27)
+				)
+				(justify left)
 			)
 		)
@@
 	(global_label "Fan2"
 		(shape output)
-		(at 234.95 143.51 0)
-		(fields_autoplaced yes)
-		(effects
-			(font
-				(size 1.27 1.27)
-			)
-			(justify left)
-		)
-		(property "Intersheetrefs" "${INTERSHEET_REFS}"
-			(at 242.5313 143.51 0)
+		(at 234.95 146.05 0)
+		(fields_autoplaced yes)
+		(effects
+			(font
+				(size 1.27 1.27)
+			)
+			(justify left)
+		)
+		(property "Intersheetrefs" "${INTERSHEET_REFS}"
+			(at 242.5313 146.05 0)
 			(hide yes)
 			(show_name no)
@@
 		)
 	)
+	(global_label "PC6"
+		(shape bidirectional)
+		(at 199.39 161.29 180)
+		(fields_autoplaced yes)
+		(effects
+			(font
+				(size 1.27 1.27)
+			)
+			(justify right)
+		)
+		(property "Intersheetrefs" "${INTERSHEET_REFS}"
+			(at 191.544 161.29 0)
+			(hide yes)
+			(show_name no)
+			(do_not_autoplace no)
+			(effects
+				(font
+					(size 1.27 1.27)
+				)
+				(justify right)
+			)
+		)
+	)
 	(global_label "Bottom_Heater"
 		(shape output)
@@
 	(global_label "TC2_CJ_TEMP"
 		(shape input)
-		(at 234.95 135.89 0)
-		(fields_autoplaced yes)
-		(effects
-			(font
-				(size 1.27 1.27)
-			)
-			(justify left)
-		)
-		(property "Intersheetrefs" "${INTERSHEET_REFS}"
-			(at 248.454 135.89 0)
+		(at 234.95 125.73 0)
+		(fields_autoplaced yes)
+		(effects
+			(font
+				(size 1.27 1.27)
+			)
+			(justify left)
+		)
+		(property "Intersheetrefs" "${INTERSHEET_REFS}"
+			(at 248.454 125.73 0)
 			(hide yes)
 			(show_name no)
@@
 	(global_label "Fan1"
 		(shape output)
-		(at 234.95 148.59 0)
-		(fields_autoplaced yes)
-		(effects
-			(font
-				(size 1.27 1.27)
-			)
-			(justify left)
-		)
-		(property "Intersheetrefs" "${INTERSHEET_REFS}"
-			(at 242.5313 148.59 0)
+		(at 234.95 143.51 0)
+		(fields_autoplaced yes)
+		(effects
+			(font
+				(size 1.27 1.27)
+			)
+			(justify left)
+		)
+		(property "Intersheetrefs" "${INTERSHEET_REFS}"
+			(at 242.5313 143.51 0)
 			(hide yes)
 			(show_name no)
@@
 		)
 	)
+	(global_label "PB14"
+		(shape bidirectional)
+		(at 237.49 194.31 0)
+		(fields_autoplaced yes)
+		(effects
+			(font
+				(size 1.27 1.27)
+			)
+			(justify left)
+		)
+		(property "Intersheetrefs" "${INTERSHEET_REFS}"
+			(at 246.5455 194.31 0)
+			(hide yes)
+			(show_name no)
+			(do_not_autoplace no)
+			(effects
+				(font
+					(size 1.27 1.27)
+				)
+				(justify left)
+			)
+		)
+	)
+	(global_label "PB12"
+		(shape bidirectional)
+		(at 234.95 189.23 0)
+		(fields_autoplaced yes)
+		(effects
+			(font
+				(size 1.27 1.27)
+			)
+			(justify left)
+		)
+		(property "Intersheetrefs" "${INTERSHEET_REFS}"
+			(at 244.0055 189.23 0)
+			(hide yes)
+			(show_name no)
+			(do_not_autoplace no)
+			(effects
+				(font
+					(size 1.27 1.27)
+				)
+				(justify left)
+			)
+		)
+	)
 	(global_label "TC1_CJ_TEMP"
 		(shape input)
@@
 	(global_label "TC1_ADC"
 		(shape input)
-		(at 234.95 130.81 0)
-		(fields_autoplaced yes)
-		(effects
-			(font
-				(size 1.27 1.27)
-			)
-			(justify left)
-		)
-		(property "Intersheetrefs" "${INTERSHEET_REFS}"
-			(at 244.5481 130.81 0)
-			(hide yes)
-			(show_name no)
-			(do_not_autoplace no)
-			(effects
-				(font
-					(size 1.27 1.27)
-				)
-				(justify left)
-			)
-		)
-	)
-	(global_label "PB2"
-		(shape output)
-		(at 237.49 166.37 0)
-		(fields_autoplaced yes)
-		(effects
-			(font
-				(size 1.27 1.27)
-			)
-			(justify left)
-		)
-		(property "Intersheetrefs" "${INTERSHEET_REFS}"
-			(at 244.2247 166.37 0)
+		(at 234.95 135.89 0)
+		(fields_autoplaced yes)
+		(effects
+			(font
+				(size 1.27 1.27)
+			)
+			(justify left)
+		)
+		(property "Intersheetrefs" "${INTERSHEET_REFS}"
+			(at 245.9785 135.89 0)
+			(hide yes)
+			(show_name no)
+			(do_not_autoplace no)
+			(effects
+				(font
+					(size 1.27 1.27)
+				)
+				(justify left)
+			)
+		)
+	)
+	(global_label "PB15"
+		(shape bidirectional)
+		(at 237.49 196.85 0)
+		(fields_autoplaced yes)
+		(effects
+			(font
+				(size 1.27 1.27)
+			)
+			(justify left)
+		)
+		(property "Intersheetrefs" "${INTERSHEET_REFS}"
+			(at 246.5455 196.85 0)
+			(hide yes)
+			(show_name no)
+			(do_not_autoplace no)
+			(effects
+				(font
+					(size 1.27 1.27)
+				)
+				(justify left)
+			)
+		)
+	)
+	(global_label "PB13"
+		(shape bidirectional)
+		(at 234.95 191.77 0)
+		(fields_autoplaced yes)
+		(effects
+			(font
+				(size 1.27 1.27)
+			)
+			(justify left)
+		)
+		(property "Intersheetrefs" "${INTERSHEET_REFS}"
+			(at 244.0055 191.77 0)
 			(hide yes)
 			(show_name no)
@@
 	(global_label "TC2_ADC"
 		(shape input)
-		(at 234.95 128.27 0)
-		(fields_autoplaced yes)
-		(effects
-			(font
-				(size 1.27 1.27)
-			)
-			(justify left)
-		)
-		(property "Intersheetrefs" "${INTERSHEET_REFS}"
-			(at 244.5481 128.27 0)
+		(at 234.95 123.19 0)
+		(fields_autoplaced yes)
+		(effects
+			(font
+				(size 1.27 1.27)
+			)
+			(justify left)
+		)
+		(property "Intersheetrefs" "${INTERSHEET_REFS}"
+			(at 244.5481 123.19 0)
 			(hide yes)
 			(show_name no)
@@
 		)
 	)
-	(global_label "PB1"
-		(shape output)
-		(at 237.49 163.83 0)
-		(fields_autoplaced yes)
-		(effects
-			(font
-				(size 1.27 1.27)
-			)
-			(justify left)
-		)
-		(property "Intersheetrefs" "${INTERSHEET_REFS}"
-			(at 244.2247 163.83 0)
-			(hide yes)
-			(show_name no)
-			(do_not_autoplace no)
-			(effects
-				(font
-					(size 1.27 1.27)
-				)
-				(justify left)
-			)
-		)
-	)
 	(global_label "Fan3"
 		(shape output)
-		(at 234.95 146.05 0)
-		(fields_autoplaced yes)
-		(effects
-			(font
-				(size 1.27 1.27)
-			)
-			(justify left)
-		)
-		(property "Intersheetrefs" "${INTERSHEET_REFS}"
-			(at 242.5313 146.05 0)
-			(hide yes)
-			(show_name no)
-			(do_not_autoplace no)
-			(effects
-				(font
-					(size 1.27 1.27)
-				)
-				(justify left)
-			)
-		)
-	)
-	(global_label "PB0"
-		(shape output)
-		(at 237.49 161.29 0)
-		(fields_autoplaced yes)
-		(effects
-			(font
-				(size 1.27 1.27)
-			)
-			(justify left)
-		)
-		(property "Intersheetrefs" "${INTERSHEET_REFS}"
-			(at 244.2247 161.29 0)
-			(hide yes)
-			(show_name no)
+		(at 234.95 148.59 0)
+		(fields_autoplaced yes)
+		(effects
+			(font
+				(size 1.27 1.27)
+			)
+			(justify left)
+		)
+		(property "Intersheetrefs" "${INTERSHEET_REFS}"
+			(at 242.5313 148.59 0)
+			(hide yes)
+			(show_name no)

Commit message: tweak board design more
Parts:
- added R60: 10k, Resistor_SMD:R_0603_1608Metric_Pad0.98x0.95mm_HandSolder, symbol Device:R_US
- added SW4: SW_Push, Button_Switch_THT:SW_PUSH_6mm_H4.3mm, symbol Switch:SW_Push
Connections:
- net +3.3V: now also R60.1
- net GND: now also SW4.2
- net STM_USR_BTN: now reaches U4.14 (PA0)
- net STM_USR_BTN: now also R60.2, SW4.1
- no-connect marks 14 -> 13

Commit message: board tweaked, sent for review
Parts:
- SW3, SW4: footprint Button_Switch_THT:SW_PUSH_6mm_H4.3mm -> Button_Switch_THT:SW_PUSH_6mm_H8.5mm
Changed lines of the file:
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@@
 			)
 		)
-		(property "Footprint" "Button_Switch_THT:SW_PUSH_6mm_H4.3mm"
+		(property "Footprint" "Button_Switch_THT:SW_PUSH_6mm_H8.5mm"
 			(at 275.59 113.03 0)
 			(hide yes)
@@
 			)
 		)
-		(property "Footprint" "Button_Switch_THT:SW_PUSH_6mm_H4.3mm"
+		(property "Footprint" "Button_Switch_THT:SW_PUSH_6mm_H8.5mm"
 			(at 163.83 88.9 0)
 			(hide yes)
