File: mainBoard/triac.kicad_sch (KiCad schematic)
At the start: 35 parts, among them J2 1366005, J3 1366005, Q1 IRLML6244TRPBF, Q2 IRLML6244TRPBF, SW5 SW_DPST_x2, U14 DS18B20+, U15 DS18B20+, U6 MOC3083S-TA1, U7 MOC3083S-TA1

Commit message: Nearly finished with board after revisions
Parts:
- removed F2, F3: 10A, Fuse:Fuseholder_Clip-6.3x32mm_Littelfuse_122_Inline_P34.21x7.62mm_D2.54mm_Horizontal, symbol Device:Fuse
- removed SW5: SW_DPST_x2, TerminalBlock_Phoenix:TerminalBlock_Phoenix_MKDS-1,5-2-5.08_1x02_P5.08mm_Horizontal, symbol Switch:SW_DPST_x2
- C25, C26: value 10nF 250V -> 10nF; Field5 (none) -> 250V C0G
- R12, R13: value 39 -> 39 1W
- R14, R15, R16, R17: value 330 -> 330 1W
Connections:
- net L1_F3_BOT is gone; now on net L1_SW: C26.2, D7.1 (A1), R17.1
- net +5V: now also U6.1, U7.1; no longer R20.1, R21.1
- net OPTO_K_BOT: now also R21.1; no longer Q2.3 (D), R25.2
- net OPTO_K_TOP: now also R20.1; no longer Q1.3 (D), R24.2
- net L1_F2_TOP renamed L1_SW
- net LN_BOT renamed L1_BOT
- net LN_OPTO_BOT renamed L1_OPTO_BOT
- net LN_OPTO_TOP renamed L1_OPTO_TOP
- net LN_TOP renamed L1_TOP
- net OPTO_A_BOT renamed OPTO_FETD_BOT
- net OPTO_FETD_BOT: now also Q2.3 (D), R25.2; no longer U7.1
- net OPTO_A_TOP renamed OPTO_FETD_TOP
- net OPTO_FETD_TOP: now also Q1.3 (D), R24.2; no longer U6.1
- net OPTO_FET_BOT renamed OPTO_FETG_BOT
- net OPTO_FET_TOP renamed OPTO_FETG_TOP
Other:
- note removed: "StackExchange resources for TRIAC driver design"
- note removed: "https://electronics.stackexchange.com/questions/248743/how-is-the-gate-trigger-resistor-value-calculated-for-a-triac/248775"
- note removed: "https://electronics.stackexchange.com/questions/381961/triac-optocoupler-circuit"
- note removed: "https://electronics.stackexchange.com/questions/437809/triac-switching-circuit-with-optocoupler"
- note removed: "https://electronics.stackexchange.com/questions/53500/optotriactriac-how-do-i-calculate-the-gate-resistor"
- moved on the sheet: C25, D6, D7, D8, D9, HS1, HS2, J2, J3, Q1, Q2, R12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

Commit message: work on AC power side
Parts:
- removed J2, J3: 1366005, PhoenixContact_SPTA:SPTA-THR 2.53-5.0 P26, symbol Connector_Generic:Conn_01x03
- added J14, J18: 1714971, PhoenixContact_MKDS_9mm:CONN_1714971_PXC, symbol Connector_Generic:Conn_01x02
Connections:
- net L1_BOT: now also J14.2 (Pin_2)
- net L1_TOP: now also J18.2 (Pin_2)
- net LN: now also J14.1 (Pin_1), J18.1 (Pin_1)
Changed lines of the file:
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@@
 	)
 	(junction
-		(at 186.69 90.17)
-		(diameter 0)
-		(color 0 0 0 0)
-	)
-	(junction
 		(at 290.83 162.56)
 		(diameter 0)
@@
 	)
 	(junction
+		(at 186.69 162.56)
+		(diameter 0)
+		(color 0 0 0 0)
+	)
+	(junction
 		(at 350.52 199.39)
 		(diameter 0)
@@
 	)
 	(junction
+		(at 186.69 90.17)
+		(diameter 0)
+		(color 0 0 0 0)
+	)
+	(junction
 		(at 186.69 186.69)
 		(diameter 0)
@@
 	)
 	(junction
-		(at 186.69 162.56)
-		(diameter 0)
-		(color 0 0 0 0)
-	)
-	(junction
 		(at 213.36 186.69)
 		(diameter 0)
@@
 	(wire
 		(pts
-			(xy 148.59 162.56) (xy 186.69 162.56)
+			(xy 146.05 162.56) (xy 186.69 162.56)
 		)
 		(stroke
@@
 	(wire
 		(pts
-			(xy 147.32 85.09) (xy 147.32 90.17)
+			(xy 144.78 85.09) (xy 144.78 90.17)
 		)
 		(stroke
@@
 	(wire
 		(pts
-			(xy 147.32 90.17) (xy 186.69 90.17)
+			(xy 144.78 90.17) (xy 186.69 90.17)
 		)
 		(stroke
@@
 	(wire
 		(pts
-			(xy 148.59 157.48) (xy 148.59 162.56)
+			(xy 146.05 157.48) (xy 146.05 162.56)
 		)
 		(stroke
@@
 	(wire
 		(pts
-			(xy 144.78 85.09) (xy 144.78 92.71)
-		)
-		(stroke
-			(width 0)
-			(type default)
-		)
-	)
-	(wire
-		(pts
 			(xy 213.36 92.71) (xy 213.36 90.17)
 		)
@@
 	(wire
 		(pts
-			(xy 146.05 157.48) (xy 146.05 165.1)
-		)
-		(stroke
-			(width 0)
-			(type default)
-		)
-	)
-	(wire
-		(pts
 			(xy 267.97 95.25) (xy 267.97 104.14)
 		)
@@
 	)
 	(symbol
-		(lib_id "Connector_Generic:Conn_01x03")
-		(at 144.78 80.01 270)
-		(mirror x)
+		(lib_id "Connector_Generic:Conn_01x02")
+		(at 143.51 152.4 90)
 		(unit 1)
 		(body_style 1)
@@
 		(in_pos_files yes)
 		(dnp no)
-		(property "Reference" "J2"
-			(at 139.7 78.7399 90)
+		(fields_autoplaced yes)
+		(property "Reference" "J14"
+			(at 148.59 151.13 90)
 			(show_name no)
 			(do_not_autoplace no)
@@
 			)
 		)
-		(property "Value" "1366005"
-			(at 139.7 81.2799 90)
+		(property "Value" "1714971"
+			(at 148.59 153.67 90)
 			(show_name no)
 			(do_not_autoplace no)
@@
 			)
 		)
-		(property "Footprint" "PhoenixContact_SPTA:SPTA-THR 2.53-5.0 P26"
-			(at 144.78 80.01 0)
+		(property "Footprint" "PhoenixContact_MKDS_9mm:CONN_1714971_PXC"
+			(at 143.51 152.4 0)
 			(hide yes)
 			(show_name no)
@@
 		)
 		(property "Datasheet" ""
-			(at 144.78 80.01 0)
+			(at 143.51 152.4 0)
 			(hide yes)
 			(show_name no)
@@
 			)
 		)
-		(property "Description" "Generic connector, single row, 01x03, script generated (kicad-library-utils/schlib/autogen/connector/)"
-			(at 144.78 80.01 0)
+		(property "Description" "Generic connector, single row, 01x02, script generated (kicad-library-utils/schlib/autogen/connector/)"
+			(at 143.51 152.4 0)
 			(hide yes)
 			(show_name no)
@@
 			)
 		)
-		(pin "3"
-		)
 		(pin "1"
 		)
@@
 			(project "mainBoard"
 				(path "/0650c7a8-acba-429c-9f8e-eec0baf0bc1c/fede4c36-00cc-4d3d-b71c-5243ba232202/db0f358e-afa6-42f8-adbe-74e998d63224"
-					(reference "J2")
+					(reference "J14")
 					(unit 1)
 				)
@@
 	)
 	(symbol
-		(lib_id "power:GNDPWR")
-		(at 144.78 92.71 0)
-		(mirror y)
-		(unit 1)
-		(body_style 1)
-		(exclude_from_sim no)
-		(in_bom yes)
-		(on_board yes)
-		(in_pos_files yes)
-		(dnp no)
-		(fields_autoplaced yes)
-		(property "Reference" "#PWR036"
-			(at 144.78 97.79 0)
-			(hide yes)
-			(show_name no)
-			(do_not_autoplace no)
-			(effects
-				(font
-					(size 1.27 1.27)
-				)
-			)
-		)
-		(property "Value" "GNDPWR"
-			(at 144.907 96.52 0)
-			(hide yes)
-			(show_name no)
-			(do_not_autoplace no)
-			(effects
-				(font
-					(size 1.27 1.27)
-				)
-			)
-		)
-		(property "Footprint" ""
-			(at 144.78 93.98 0)
-			(hide yes)
-			(show_name no)
-			(do_not_autoplace no)
-			(effects
-				(font
-					(size 1.27 1.27)
-				)
-			)
-		)
-		(property "Datasheet" ""
-			(at 144.78 93.98 0)
-			(hide yes)
-			(show_name no)
-			(do_not_autoplace no)
-			(effects
-				(font
-					(size 1.27 1.27)
-				)
-			)
-		)
-		(property "Description" "Power symbol creates a global label with name \"GNDPWR\" , global ground"
-			(at 144.78 92.71 0)
-			(hide yes)
-			(show_name no)
-			(do_not_autoplace no)
-			(effects
-				(font
-					(size 1.27 1.27)
-				)
-			)
-		)
-		(pin "1"
-		)
-		(instances
-			(project "mainBoard"
-				(path "/0650c7a8-acba-429c-9f8e-eec0baf0bc1c/fede4c36-00cc-4d3d-b71c-5243ba232202/db0f358e-afa6-42f8-adbe-74e998d63224"
-					(reference "#PWR036")
-					(unit 1)
-				)
-			)
-		)
-	)
-	(symbol
 		(lib_id "power:+5V")
 		(at 290.83 154.94 0)
@@
 	)
 	(symbol
-		(lib_id "Connector_Generic:Conn_01x03")
-		(at 146.05 152.4 270)
-		(mirror x)
+		(lib_id "Connector_Generic:Conn_01x02")
+		(at 142.24 80.01 90)
 		(unit 1)
 		(body_style 1)
@@
 		(in_pos_files yes)
 		(dnp no)
-		(property "Reference" "J3"
-			(at 140.97 151.1299 90)
+		(fields_autoplaced yes)
+		(property "Reference" "J18"
+			(at 147.32 78.74 90)
 			(show_name no)
 			(do_not_autoplace no)
@@
 			)
 		)
-		(property "Value" "1366005"
-			(at 140.97 153.6699 90)
+		(property "Value" "1714971"
+			(at 147.32 81.28 90)
 			(show_name no)
 			(do_not_autoplace no)
@@
 			)
 		)
-		(property "Footprint" "PhoenixContact_SPTA:SPTA-THR 2.53-5.0 P26"
-			(at 146.05 152.4 0)
+		(property "Footprint" "PhoenixContact_MKDS_9mm:CONN_1714971_PXC"
+			(at 142.24 80.01 0)
 			(hide yes)
 			(show_name no)
@@
 		)
 		(property "Datasheet" ""
-			(at 146.05 152.4 0)
+			(at 142.24 80.01 0)
 			(hide yes)
 			(show_name no)
@@
 			)
 		)
-		(property "Description" "Generic connector, single row, 01x03, script generated (kicad-library-utils/schlib/autogen/connector/)"
-			(at 146.05 152.4 0)
+		(property "Description" "Generic connector, single row, 01x02, script generated (kicad-library-utils/schlib/autogen/connector/)"
+			(at 142.24 80.01 0)
 			(hide yes)
 			(show_name no)
@@
 			)
 		)
-		(pin "3"
-		)
 		(pin "1"
 		)
@@
 			(project "mainBoard"
 				(path "/0650c7a8-acba-429c-9f8e-eec0baf0bc1c/fede4c36-00cc-4d3d-b71c-5243ba232202/db0f358e-afa6-42f8-adbe-74e998d63224"
-					(reference "J3")
+					(reference "J18")
 					(unit 1)
 				)
@@
 					(unit 1)
 				)
-			)
-		)
-	)
-	(symbol
-		(lib_id "power:GNDPWR")
-		(at 146.05 165.1 0)
-		(mirror y)
-		(unit 1)
-		(body_style 1)
-		(exclude_from_sim no)
-		(in_bom yes)
-		(on_board yes)
-		(in_pos_files yes)
-		(dnp no)
-		(fields_autoplaced yes)
-		(property "Reference" "#PWR037"
-			(at 146.05 170.18 0)
-			(hide yes)
-			(show_name no)
-			(do_not_autoplace no)
-			(effects
-				(font
-					(size 1.27 1.27)
-				)
-			)
-		)
-		(property "Value" "GNDPWR"
-			(at 146.177 168.91 0)
-			(hide yes)
-			(show_name no)
-			(do_not_autoplace no)
-			(effects
-				(font
-					(size 1.27 1.27)
-				)
-			)
-		)
-		(property "Footprint" ""
-			(at 146.05 166.37 0)
-			(hide yes)
-			(show_name no)
-			(do_not_autoplace no)
-			(effects
-				(font
-					(size 1.27 1.27)
-				)
-			)
-		)
-		(property "Datasheet" ""
-			(at 146.05 166.37 0)
-			(hide yes)
-			(show_name no)
-			(do_not_autoplace no)
-			(effects
-				(font
-					(size 1.27 1.27)
-				)
-			)
-		)
-		(property "Description" "Power symbol creates a global label with name \"GNDPWR\" , global ground"
-			(at 146.05 165.1 0)
-			(hide yes)
-			(show_name no)
-			(do_not_autoplace no)
-			(effects
-				(font
-					(size 1.27 1.27)
-				)
-			)
-		)
-		(pin "1"
-		)
-		(instances
-			(project "mainBoard"
-				(path "/0650c7a8-acba-429c-9f8e-eec0baf0bc1c/fede4c36-00cc-4d3d-b71c-5243ba232202/db0f358e-afa6-42f8-adbe-74e998d63224"
-					(reference "#PWR037")
-					(unit 1)
-				)
