File: mainBoard/thermocouple.kicad_sch (KiCad schematic)
At the start: 60 parts, among them J4 4DB-P108-02, J5 4DB-P108-02, J6 4DB-P108-02, U10 DS18B20+, U11 DS18B20+, U12 OPA333AIDCKT, U13 DS18B20+, U8 OPA333AIDCKT, U9 OPA333AIDCKT

Commit message: Nearly finished with board after revisions
Parts:
- removed TP10, TP11, TP12, TP15, TP16, TP7: TestPoint, TestPoint:TestPoint_Keystone_5019_Miniature, symbol Connector:TestPoint
- C27, C28, C35: value 1uF C0G -> 1uF; Type (none) -> 6.3V C0G
- C29, C30, C36: value 100nF C0G -> 100nF; footprint Capacitor_SMD:C_0805_2012Metric_Pad1.18x1.45mm_HandSolder -> Capacitor_SMD:C_0603_1608Metric_Pad1.08x0.95mm_HandSolder; Type (none) -> 6.3V C0G
- C33: value 10uF C0G -> 10uF; Type (none) -> 6.3V C0G
- TP13, TP14, TP5, TP6, TP8, TP9: footprint TestPoint:TestPoint_Keystone_5019_Miniature -> TestPoint:TestPoint_Pad_D1.5mm
Connections:
- net TC1_N: now also J4.2 (Pin_2); no longer J4.1 (Pin_1)
- net TC1_P: now also J4.1 (Pin_1); no longer J4.2 (Pin_2)
- net TC2_N: now also J5.2 (Pin_2); no longer J5.1 (Pin_1)
- net TC2_P: now also J5.1 (Pin_1); no longer J5.2 (Pin_2)
- net TC3_N: now also J6.2 (Pin_2); no longer J6.1 (Pin_1)
- net TC3_P: now also J6.1 (Pin_1); no longer J6.2 (Pin_2)
Other:
- note added: "Channel 1"
- note added: "Channel 2"
- note added: "Channel 3"
- moved on the sheet: C27, C31, C32, C34, C37, C38, J4, J5, J6, JP5, JP6, JP7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

Commit message: change to single 4" touchscreen for UI instead of keypad and buttons
Parts:
- renumbered C27 to C34, C28 to C35, C29 to C36, C30 to C37, C31 to C38, C32 to C39, C33 to C40, C38 to C41, C35 to C42, C36 to C43, C37 to C44, C34 to C45, J4 to J5, J5 to J6, J6 to J7, JP7 to JP10, JP5 to JP8, JP6 to JP9, R26 to R41, R27 to R42, R28 to R43, R29 to R44, R30 to R45, R31 to R46, R32 to R47, R33 to R48, R34 to R49, R35 to R50, R36 to R51, R37 to R52, R66 to R53, R68 to R54, R38 to R55, R46 to R56, R40 to R57, R41 to R58, R42 to R59, R43 to R60, R44 to R61, R45 to R62, R67 to R63, R39 to R64, TP5 to TP16, TP6 to TP17, TP8 to TP18, TP9 to TP19, TP13 to TP20, TP14 to TP21, U8 to U11, U9 to U12, U10 to U13, U11 to U14, U12 to U15, U13 to U16
