File: mainBoard/_autosave-mcu.kicad_sch (KiCad schematic)
At the start: 36 parts, among them J2 USB_A, SW2 SW_SPDT, SW3 SW_Push, SW4 SW_Push, U19 23LC1024-I/ST, U5 USBLC6-2SC6, U6 STM32F413RHT6, Y1 RH100-48.000-10-F-1015-X-TR-N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

Commit message: working on layout
Parts:
- added J16: Conn_01x04, Connector_JST:JST_XH_B2B-XH-A_1x04_P2.50mm_Vertical, symbol Connector_Generic:Conn_01x04
Connections:
- net GND: now also J16.3 (Pin_3), J16.4 (Pin_4)
- new net +5V: J16.1 (Pin_1)
Other:
- note added: "JST XH"
- note added: "WS2812B LED Strip"
