File: mainBoard/_autosave-mainBoard.kicad_pcb (KiCad board)
At the start: 4 copper layers, 274.8 x 176.1 mm, 302 parts, among them J1 1366005, J10 Conn_01x02, J11 Conn_02x05_Odd_Even, J12 Conn_01x02, J13 Conn_01x02, J14 Conn_01x06, J15 Conn_01x03, J17 Conn_01x05, J18 Conn_01x04, J19 Conn_01x14, J2 USB_A, J3 1714971, J4 1714971, J5 4DB-P108-02, J6 4DB-P108-02, J7 4DB-P108-02, J8 Conn_01x02, J9 Conn_01x02, K1 Relay_SPDT, Q1 IRLML6244TRPBF, Q2 IRLML6244TRPBF, Q3 IRLML6244TRPBF, Q4 IRLML6244TRPBF, Q5 IRLML6244TRPBF, Q7 IRLML6244TRPBF, Q8 PMOS, SW1 SW_SPST, SW2 SW_SPDT, SW3 SW_Push, SW4 SW_Push, U1 RT6255BHGJ8F, U10 DS18B20+, U11 OPA333AIDCKT, U12 OPA333AIDCKT, U13 DS18B20+, U14 DS18B20+, U15 OPA333AIDCKT, U16 DS18B20+, U17 SFH617A-2, U18 USBLC6-4SC6, U19 23LC1024-E/SN, U2 RT9059GSP, U20 LM386, U21 USBLC6-4SC6, U22 W25Q128JVSIQ TR, U23 USBLC6-4SC6, U24 USBLC6-2SC6, U26 100, U27 100, U28 100, U29 100, U3 RT9059GSP, U30 74LVC1T45W6-7, U32 74LVC1T45W6-7, U4 TPS2041B, U5 USBLC6-2SC6, U6 STM32F413RHT6, U7 MOC3083S-TA1, U8 MOC3083S-TA1, U9 DS18B20+, Y1 RH100-48.000-10-F-1015-X-TR-N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

Commit message: remove dual ESD protection on nRST and route nrst to stlink
Routing:
- net NRST_SW: track 162.6 -> 152.7 mm
Changed lines of the file:
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@@
-	)
-	(segment
-		(start 262.300002 136.2)
-		(end 262.300002 135.537501)
-		(width 0.3)
-		(layer "F.Cu")
-		(net "NRST_SW")
 	)
 	(segment
@@
 		(end 294.3 131.3)
 		(width 0.2)
-		(layer "F.Cu")
-		(net "NRST_SW")
-	)
-	(segment
-		(start 262.300002 135.537501)
-		(end 262.737503 135.1)
-		(width 0.3)
 		(layer "F.Cu")
 		(net "NRST_SW")
@@
 	)
 	(segment
-		(start 266.4 135.1)
-		(end 269.9 131.6)
-		(width 0.3)
-		(layer "F.Cu")
-		(net "NRST_SW")
-	)
-	(segment
 		(start 274.3 118.8625)
 		(end 274.3 120.799999)
@@
 		(layer "F.Cu")
 		(net "NRST_SW")
-	)
-	(segment
-		(start 262.737503 135.1)
-		(end 266.4 135.1)
-		(width 0.3)
-		(layer "F.Cu")
-		(net "NRST_SW")
